Commit message: refactor: Refactor DLIO launch to use a shared stack with external geometry, update sensor x-coordinates, and increase camera resolutions.

File: urdf/ig_handle_sensors.urdf.xacro (robot description, xacro)
@@ -112,5 +112,5 @@
     <parent link="base_link"/>
     <child link="lidar_v_mount"/>
-    <origin xyz="-0.180 0.126 0.11" rpy="0 0 0"/>
+    <origin xyz="0.180 0.126 0.11" rpy="0 0 0"/>
   </joint>
   <link name="lidar_v_link">
@@ -127,6 +127,6 @@
     <parent link="base_link"/>
     <child link="lidar_v_link"/>
-    <!-- X negated, rotated 90deg pitch for vertical scanning -->
-    <origin xyz="-0.180 0.126 0.181" rpy="0 1.5708 0"/>
+    <!-- Rotated 90deg pitch for vertical scanning -->
+    <origin xyz="0.180 0.126 0.181" rpy="0 1.5708 0"/>
   </joint>
   <gazebo reference="lidar_v_link">
@@ -241,5 +241,5 @@
     <parent link="base_link"/>
     <child link="camera_mount"/>
-    <origin xyz="-0.0164 0.1 0.13" rpy="0 0 0"/>
+    <origin xyz="0.0164 0.1 0.13" rpy="0 0 0"/>
   </joint>
   <!-- ====================================================================== -->
@@ -260,5 +260,5 @@
     <parent link="base_link"/>
     <child link="camera_F1_link"/>
-    <origin xyz="-0.0164 0.0213 0.230" rpy="0 0 0"/>
+    <origin xyz="0.0164 0.0213 0.230" rpy="0 0 0"/>
   </joint>
   <link name="camera_F1_optical_link"/>
@@ -274,6 +274,6 @@
         <horizontal_fov>1.60</horizontal_fov>
         <image>
-          <width>640</width>
-          <height>480</height>
+          <width>1280</width>
+          <height>1024</height>
           <format>R8G8B8</format>
         </image>
@@ -321,5 +321,5 @@
     <parent link="base_link"/>
     <child link="camera_F2_link"/>
-    <origin xyz="-0.0164 0.2033 0.230" rpy="0 0 0"/>
+    <origin xyz="0.0164 0.2033 0.230" rpy="0 0 0"/>
   </joint>
   <link name="camera_F2_optical_link"/>
@@ -335,6 +335,6 @@
         <horizontal_fov>1.60</horizontal_fov>
         <image>
-          <width>640</width>
-          <height>480</height>
+          <width>1280</width>
+          <height>1024</height>
           <format>R8G8B8</format>
         </image>
@@ -384,5 +384,5 @@
     <parent link="base_link"/>
     <child link="debug_extra_link"/>
-    <origin xyz="-0.0656 0.091 0.203" rpy="0 0 0"/>
+    <origin xyz="0.0656 0.091 0.203" rpy="0 0 0"/>
   </joint>
   <gazebo>
