Commit message: Refactor: Switch to kinematic planarmove simulation, fix visual meshes, and remove unstable physics plugins

File: urdf/heron_sim.urdf.xacro (robot description, xacro)
@@ -32,10 +32,11 @@
   <!-- Heron Base Link (Hull) -->
   <!-- ====================================================================== -->
+  <!-- Heron Base Link (Hull) -->
   <link name="base_link">
     <visual>
       <geometry>
-        <box size="1.35 1.0 0.25"/>
-      </geometry>
-      <origin xyz="0 0 0.05" rpy="0 0 0"/>
+        <mesh filename="package://heron_description/meshes/heron_base.stl" scale="1 1 1"/>
+      </geometry>
+      <origin xyz="0 0 0" rpy="0 0 0"/>
       <material name="heron_grey"/>
     </visual>
@@ -56,7 +57,8 @@
     <visual>
       <geometry>
-        <box size="1.2 0.2 0.15"/>
+        <mesh filename="package://heron_description/meshes/left_panel.stl" scale="1 1 1"/>
       </geometry>
       <material name="heron_yellow"/>
+      <origin xyz="0 0 0" rpy="0 0 0"/>
     </visual>
     <inertial>
@@ -68,5 +70,5 @@
     <parent link="base_link"/>
     <child link="left_pontoon"/>
-    <origin xyz="0 0.4 -0.05" rpy="0 0 0"/>
+    <origin xyz="0 0.34495 0.04959" rpy="0 0 0"/>
   </joint>
   <!-- Right pontoon (visual only) -->
@@ -74,7 +76,8 @@
     <visual>
       <geometry>
-        <box size="1.2 0.2 0.15"/>
+        <mesh filename="package://heron_description/meshes/right_panel.stl" scale="1 1 1"/>
       </geometry>
       <material name="heron_yellow"/>
+      <origin xyz="0 0 0" rpy="0 0 0"/>
     </visual>
     <inertial>
@@ -86,5 +89,5 @@
     <parent link="base_link"/>
     <child link="right_pontoon"/>
-    <origin xyz="0 -0.4 -0.05" rpy="0 0 0"/>
+    <origin xyz="0 -0.34495 0.04959" rpy="0 0 0"/>
   </joint>
   <!-- ====================================================================== -->
@@ -381,5 +384,5 @@
     <sensor type="ray" name="lidar_h_sensor">
       <pose>0 0 0 0 0 0</pose>
-      <visualize>true</visualize>
+      <visualize>false</visualize>
       <update_rate>10</update_rate>
       <ray>
@@ -421,5 +424,5 @@
     <sensor type="ray" name="lidar_v_sensor">
       <pose>0 0 0 1.5708 0 0</pose>
-      <visualize>true</visualize>
+      <visualize>false</visualize>
       <update_rate>10</update_rate>
       <ray>

Commit message: chore: sync changes

File: urdf/heron_sim.urdf.xacro (robot description, xacro)
@@ -32,5 +32,10 @@
   <!-- Heron Base Link (Hull) -->
   <!-- ====================================================================== -->
-  <!-- Heron Base Link (Hull) -->
+  <link name="base_footprint"/>
+  <joint name="base_footprint_joint" type="fixed">
+    <origin xyz="0 0 0" rpy="0 0 0" />
+    <parent link="base_footprint" />
+    <child link="base_link" />
+  </joint>
   <link name="base_link">
     <visual>
@@ -412,7 +417,12 @@
         </noise>
       </ray>
-      <plugin name="lidar_h_plugin" filename="libgazebo_ros_laser.so">
+      <plugin name="lidar_h_plugin" filename="libgazebo_ros_velodyne_laser.so">
         <topicName>/lidar_h/velodyne_points</topicName>
         <frameName>lidar_h_link</frameName>
+        <min_range>1.2</min_range>
+        <max_range>130.0</max_range>
+        <gaussianNoise>0.01</gaussianNoise>
+        <min_intensity>0.0</min_intensity>
+        <organize_cloud>true</organize_cloud>
       </plugin>
     </sensor>
@@ -449,4 +459,9 @@
         <topicName>/lidar_v/velodyne_points</topicName>
         <frameName>lidar_v_link</frameName>
+        <min_range>1.2</min_range>
+        <max_range>130.0</max_range>
+        <gaussianNoise>0.01</gaussianNoise>
+        <min_intensity>0.0</min_intensity>
+        <organize_cloud>true</organize_cloud>
       </plugin>
     </sensor>
@@ -544,4 +559,5 @@
       <robotBaseFrame>base_link</robotBaseFrame>
       <publishOdomTF>false</publishOdomTF>
+      <cmdTimeout>-1.0</cmdTimeout>
     </plugin>
   </gazebo>

Commit message: feat: Update vessel dynamics parameters, integrate IMU and sonar sensors, and refactor existing lidar and camera configurations with new topic names for improved simulation realism.

File: urdf/heron_sim.urdf.xacro (robot description, xacro)
@@ -53,7 +53,7 @@
     </collision>
     <inertial>
-      <mass value="30.0"/>
-      <origin xyz="0 0 0" rpy="0 0 0"/>
-      <inertia ixx="2.5" ixy="0" ixz="0" iyy="4.5" iyz="0" izz="5.5"/>
+      <mass value="38.0"/>
+      <origin xyz="0 0 0" rpy="0 0 0"/>
+      <inertia ixx="3.4" ixy="0" ixz="0" iyy="6.0" iyz="0" izz="9.0"/>
     </inertial>
   </link>
@@ -118,4 +118,18 @@
     <origin xyz="0.0656 0.091 0.203" rpy="0 0 0"/>
   </joint>
+  <gazebo>
+    <plugin name="imu_controller" filename="libhector_gazebo_ros_imu.so">
+      <updateRate>50.0</updateRate>
+      <bodyName>imu_link</bodyName>
+      <frameId>imu_link</frameId>
+      <topicName>/sensors/imu/data</topicName>
+      <accelDrift>0.005 0.005 0.005</accelDrift>
+      <accelGaussianNoise>0.005 0.005 0.005</accelGaussianNoise>
+      <rateDrift>0.005 0.005 0.005 </rateDrift>
+      <rateGaussianNoise>0.005 0.005 0.005 </rateGaussianNoise>
+      <headingDrift>0.005</headingDrift>
+      <headingGaussianNoise>0.005</headingGaussianNoise>
+    </plugin>
+  </gazebo>
   <!-- ====================================================================== -->
   <!-- GPS/NavSat link (same position as IMU for now) -->
@@ -332,4 +346,38 @@
     <origin xyz="0 0 -0.08" rpy="0 0 0"/>
   </joint>
+  <gazebo reference="sonar_link">
+    <sensor type="ray" name="sonar">
+      <update_rate>10</update_rate>
+      <ray>
+         <scan>
+            <horizontal>
+               <samples>3</samples>
+               <resolution>1</resolution>
+               <min_angle>-0.1</min_angle>
+               <max_angle>0.1</max_angle>
+            </horizontal>
+            <vertical>
+               <samples>3</samples>
+               <resolution>1</resolution>
+               <min_angle>-0.1</min_angle>
+               <max_angle>0.1</max_angle>
+            </vertical>
+         </scan>
+         <range>
+            <min>0.2</min>
+            <max>50.0</max>
+            <resolution>0.01</resolution>
+         </range>
+      </ray>
+      <plugin name="gazebo_ros_range" filename="libgazebo_ros_range.so">
+        <topicName>/sensors/sonar/scan</topicName>
+        <frameName>sonar_link</frameName>
+        <radiation>ultrasound</radiation>
+        <fov>0.5</fov>
+        <gaussianNoise>0.005</gaussianNoise>
+        <updateRate>10</updateRate>
+      </plugin>
+    </sensor>
+  </gazebo>
   <!-- ====================================================================== -->
   <!-- Debug/Extra Links (for compatibility) -->
@@ -400,8 +448,8 @@
           </horizontal>
           <vertical>
-            <samples>32</samples>
+            <samples>16</samples>
             <resolution>1</resolution>
-            <min_angle>-0.436</min_angle> <!-- -25 deg -->
-            <max_angle>0.261</max_angle>  <!-- +15 deg -->
+            <min_angle>-0.261799</min_angle> <!-- -15 deg -->
+            <max_angle>0.261799</max_angle>  <!-- +15 deg -->
           </vertical>
         </scan>
@@ -418,11 +466,10 @@
       </ray>
       <plugin name="lidar_h_plugin" filename="libgazebo_ros_velodyne_laser.so">
-        <topicName>/lidar_h/velodyne_points</topicName>
+        <topicName>/sensors/lidar/hori/points</topicName>
         <frameName>lidar_h_link</frameName>
-        <min_range>1.2</min_range>
+        <min_range>0.1</min_range>
         <max_range>130.0</max_range>
-        <gaussianNoise>0.01</gaussianNoise>
+        <gaussianNoise>0.005</gaussianNoise>
         <min_intensity>0.0</min_intensity>
-        <organize_cloud>true</organize_cloud>
       </plugin>
     </sensor>
@@ -439,9 +486,15 @@
         <scan>
           <horizontal>
-            <samples>180</samples>
+            <samples>360</samples>
             <resolution>1</resolution>
-            <min_angle>-1.5708</min_angle>
-            <max_angle>1.5708</max_angle>
+            <min_angle>-3.14159</min_angle>
+            <max_angle>3.14159</max_angle>
           </horizontal>
+          <vertical>
+            <samples>16</samples>
+            <resolution>1</resolution>
+            <min_angle>-0.261799</min_angle>
+            <max_angle>0.261799</max_angle>
+          </vertical>
         </scan>
         <range>
@@ -457,11 +510,9 @@
       </ray>
       <plugin name="lidar_v_plugin" filename="libgazebo_ros_velodyne_laser.so">
-        <topicName>/lidar_v/velodyne_points</topicName>
+        <topicName>/sensors/lidar/vert/points</topicName>
         <frameName>lidar_v_link</frameName>
-        <min_range>1.2</min_range>
+        <min_range>0.1</min_range>
         <max_range>130.0</max_range>
-        <gaussianNoise>0.01</gaussianNoise>
-        <min_intensity>0.0</min_intensity>
-        <organize_cloud>true</organize_cloud>
+        <gaussianNoise>0.005</gaussianNoise>
       </plugin>
     </sensor>
@@ -493,5 +544,5 @@
         <alwaysOn>true</alwaysOn>
         <updateRate>30.0</updateRate>
-        <cameraName>camera_F1</cameraName>
+        <cameraName>sensors/camera/f1</cameraName>
         <imageTopicName>image_raw</imageTopicName>
         <cameraInfoTopicName>camera_info</cameraInfoTopicName>
@@ -526,5 +577,5 @@
         <alwaysOn>true</alwaysOn>
         <updateRate>30.0</updateRate>
-        <cameraName>camera_F2</cameraName>
+        <cameraName>sensors/camera/f2</cameraName>
         <imageTopicName>image_raw</imageTopicName>
         <cameraInfoTopicName>camera_info</cameraInfoTopicName>
@@ -554,5 +605,5 @@
     <plugin name="object_controller" filename="libgazebo_ros_planar_move.so">
       <commandTopic>/cmd_vel</commandTopic>
-      <odometryTopic>odom</odometryTopic>
+      <odometryTopic>/state/odometry</odometryTopic>
       <odometryFrame>odom</odometryFrame>
       <odometryRate>50.0</odometryRate>
@@ -562,3 +613,14 @@
     </plugin>
   </gazebo>
+  <!-- ====================================================================== -->
+  <!-- Force plugin for external buoyancy (receives from vessel_dynamics.py) -->
+  <!-- ====================================================================== -->
+  <gazebo>
+    <plugin name="gazebo_ros_force" filename="libgazebo_ros_force.so">
+      <alwaysOn>true</alwaysOn>
+      <updateRate>50.0</updateRate>
+      <bodyName>base_link</bodyName>
+      <topicName>heron/hydro_forces</topicName>
+    </plugin>
+  </gazebo>
 </robot>

File: urdf/ig_handle_sensors.urdf.xacro (robot description, xacro)
@@ -65,4 +65,10 @@
             <max_angle>3.14159</max_angle>
           </horizontal>
+          <vertical>
+            <samples>16</samples>
+            <resolution>1</resolution>
+            <min_angle>-0.261799</min_angle> <!-- -15 deg -->
+            <max_angle>0.261799</max_angle>  <!-- +15 deg -->
+          </vertical>
         </scan>
         <range>
@@ -77,7 +83,10 @@
         </noise>
       </ray>
-      <plugin name="gazebo_ros_lidar_h_controller" filename="libgazebo_ros_laser.so">
-        <topicName>/lidar_h/scan</topicName>
+      <plugin name="gazebo_ros_lidar_h_controller" filename="libgazebo_ros_velodyne_laser.so">
+        <topicName>/sensors/lidar/hori/points</topicName>
         <frameName>lidar_h_link</frameName>
+        <min_range>0.1</min_range>
+        <max_range>100.0</max_range>
+        <gaussianNoise>0.005</gaussianNoise>
       </plugin>
     </sensor>
@@ -132,4 +141,10 @@
             <max_angle>3.14159</max_angle>
           </horizontal>
+          <vertical>
+            <samples>16</samples>
+            <resolution>1</resolution>
+            <min_angle>-0.261799</min_angle> <!-- -15 deg -->
+            <max_angle>0.261799</max_angle>  <!-- +15 deg -->
+          </vertical>
         </scan>
         <range>
@@ -144,7 +159,10 @@
         </noise>
       </ray>
-      <plugin name="gazebo_ros_lidar_v_controller" filename="libgazebo_ros_laser.so">
-        <topicName>/lidar_v/scan</topicName>
+      <plugin name="gazebo_ros_lidar_v_controller" filename="libgazebo_ros_velodyne_laser.so">
+        <topicName>/sensors/lidar/vert/points</topicName>
         <frameName>lidar_v_link</frameName>
+        <min_range>0.1</min_range>
+        <max_range>100.0</max_range>
+        <gaussianNoise>0.005</gaussianNoise>
       </plugin>
     </sensor>
@@ -194,5 +212,5 @@
       </ray>
       <plugin name="gazebo_ros_range" filename="libgazebo_ros_range.so">
-        <topicName>/sonar/scan</topicName>
+        <topicName>/sensors/sonar/scan</topicName>
         <frameName>sonar_link</frameName>
         <radiation>ultrasound</radiation>
@@ -269,5 +287,5 @@
         <alwaysOn>true</alwaysOn>
         <updateRate>0.0</updateRate>
-        <cameraName>heron/camera</cameraName>
+        <cameraName>sensors/camera/f1</cameraName>
         <imageTopicName>image_raw</imageTopicName>
         <cameraInfoTopicName>camera_info</cameraInfoTopicName>
@@ -328,3 +346,17 @@
     <origin xyz="-0.0656 0.091 0.203" rpy="0 0 0"/>
   </joint>
+  <gazebo>
+    <plugin name="imu_controller" filename="libhector_gazebo_ros_imu.so">
+      <updateRate>50.0</updateRate>
+      <bodyName>base_link</bodyName>
+      <frameId>imu_link</frameId>
+      <topicName>/sensors/imu/data</topicName>
+      <accelDrift>0.005 0.005 0.005</accelDrift>
+      <accelGaussianNoise>0.005 0.005 0.005</accelGaussianNoise>
+      <rateDrift>0.005 0.005 0.005 </rateDrift>
+      <rateGaussianNoise>0.005 0.005 0.005 </rateGaussianNoise>
+      <headingDrift>0.005</headingDrift>
+      <headingGaussianNoise>0.005</headingGaussianNoise>
+    </plugin>
+  </gazebo>
 </robot>

Commit message: Fix simulation navigation startup and model publishing

File: urdf/heron_sim.urdf.xacro (robot description, xacro)
@@ -236,5 +236,6 @@
     <parent link="base_link"/>
     <child link="lidar_v_link"/>
-    <origin xyz="0.180 0.126 0.181" rpy="0 0 0"/>
+    <!-- Rotated 90deg pitch to convert the VLP-16 into a vertical sweep. -->
+    <origin xyz="0.180 0.126 0.181" rpy="0 1.5708 0"/>
   </joint>
   <!-- ====================================================================== -->

Commit message: Use shared configs in simulation bringup

File: urdf/heron_sim.urdf.xacro (robot description, xacro)
@@ -391,8 +391,8 @@
     <origin xyz="0 0 0" rpy="0 0 0"/>
   </joint>
-  <link name="dummy_link"/>
-  <joint name="dummy_joint" type="fixed">
-    <parent link="base_link"/>
-    <child link="dummy_link"/>
+  <link name="compat_extra_link"/>
+  <joint name="compat_extra_joint" type="fixed">
+    <parent link="base_link"/>
+    <child link="compat_extra_link"/>
     <origin xyz="0 0 0" rpy="0 0 0"/>
   </joint>
