Commit message: Align simulated sensors with hardware contracts
Co-authored-by: Aaron John Sabu <aaronjs@g.ucla.edu>

File: urdf/heron_sim.urdf.xacro (robot description, xacro)
@@ -345,28 +345,28 @@
     <parent link="base_link"/>
     <child link="sonar_link"/>
-    <origin xyz="0 0 -0.08" rpy="0 0 0"/>
+    <origin xyz="0 0 -0.08" rpy="0 1.5708 0"/>
   </joint>
   <gazebo reference="sonar_link">
     <sensor type="ray" name="sonar">
-      <update_rate>10</update_rate>
+      <update_rate>20</update_rate>
       <ray>
          <scan>
             <horizontal>
-               <samples>64</samples>
+               <samples>480</samples>
                <resolution>1</resolution>
-               <min_angle>-0.523599</min_angle>
-               <max_angle>0.523599</max_angle>
+               <min_angle>-1.047198</min_angle>
+               <max_angle>1.047198</max_angle>
             </horizontal>
             <vertical>
-               <samples>12</samples>
+               <samples>1</samples>
                <resolution>1</resolution>
-               <min_angle>-0.174533</min_angle>
-               <max_angle>0.174533</max_angle>
+               <min_angle>0.0</min_angle>
+               <max_angle>0.0</max_angle>
             </vertical>
          </scan>
          <range>
-            <min>0.2</min>
-            <max>50.0</max>
-            <resolution>0.01</resolution>
+            <min>0.5</min>
+            <max>100.0</max>
+            <resolution>0.02</resolution>
          </range>
       </ray>
@@ -374,6 +374,6 @@
         <topicName>/sensors/sonar/scan</topicName>
         <frameName>sonar_link</frameName>
-        <min_range>0.2</min_range>
-        <max_range>50.0</max_range>
+        <min_range>0.5</min_range>
+        <max_range>100.0</max_range>
         <gaussianNoise>0.003</gaussianNoise>
         <organize_cloud>false</organize_cloud>
@@ -435,4 +435,5 @@
   <!-- ====================================================================== -->
   <!-- Horizontal Lidar Gazebo Plugin -->
+  <!-- Velodyne VLP-16 model: 16 channels, 360 degree sweep, 10 Hz at 600 RPM. -->
   <!-- ====================================================================== -->
   <gazebo reference="lidar_h_link">
@@ -444,5 +445,5 @@
         <scan>
           <horizontal>
-            <samples>1080</samples>
+            <samples>1800</samples>
             <resolution>1</resolution>
             <min_angle>-3.14159</min_angle>
@@ -458,5 +459,5 @@
         <range>
           <min>0.15</min>
-          <max>30.0</max>
+          <max>200.0</max>
           <resolution>0.01</resolution>
         </range>
@@ -471,5 +472,5 @@
         <frameName>lidar_h_link</frameName>
         <min_range>0.1</min_range>
-        <max_range>130.0</max_range>
+        <max_range>200.0</max_range>
         <gaussianNoise>0.005</gaussianNoise>
         <organize_cloud>false</organize_cloud>
@@ -480,4 +481,5 @@
   <!-- ====================================================================== -->
   <!-- Vertical Lidar Gazebo Plugin -->
+  <!-- Same VLP-16 model as lidar_h, mounted with a 90 degree pitch. -->
   <!-- ====================================================================== -->
   <gazebo reference="lidar_v_link">
@@ -489,5 +491,5 @@
         <scan>
           <horizontal>
-            <samples>360</samples>
+            <samples>1800</samples>
             <resolution>1</resolution>
             <min_angle>-3.14159</min_angle>
@@ -503,5 +505,5 @@
         <range>
           <min>0.1</min>
-          <max>20.0</max>
+          <max>200.0</max>
           <resolution>0.01</resolution>
         </range>
@@ -516,5 +518,5 @@
         <frameName>lidar_v_link</frameName>
         <min_range>0.1</min_range>
-        <max_range>130.0</max_range>
+        <max_range>200.0</max_range>
         <gaussianNoise>0.005</gaussianNoise>
         <organize_cloud>false</organize_cloud>
@@ -528,10 +530,10 @@
   <gazebo reference="camera_F1_link">
     <sensor type="camera" name="camera_F1">
-      <update_rate>30.0</update_rate>
+      <update_rate>15.0</update_rate>
       <camera name="F1">
-        <horizontal_fov>2.0944</horizontal_fov> <!-- 120 degree fisheye -->
+        <horizontal_fov>1.60</horizontal_fov>
         <image>
-          <width>640</width>
-          <height>480</height>
+          <width>1280</width>
+          <height>1024</height>
           <format>R8G8B8</format>
         </image>
@@ -549,5 +551,5 @@
       <plugin name="camera_F1_controller" filename="libgazebo_ros_camera.so">
         <alwaysOn>true</alwaysOn>
-        <updateRate>30.0</updateRate>
+        <updateRate>15.0</updateRate>
         <cameraName>sensors/camera/f1</cameraName>
         <imageTopicName>image_raw</imageTopicName>
@@ -562,10 +564,10 @@
   <gazebo reference="camera_F2_link">
     <sensor type="camera" name="camera_F2">
-      <update_rate>30.0</update_rate>
+      <update_rate>15.0</update_rate>
       <camera name="F2">
-        <horizontal_fov>2.0944</horizontal_fov> <!-- 120 degree fisheye -->
+        <horizontal_fov>1.60</horizontal_fov>
         <image>
-          <width>640</width>
-          <height>480</height>
+          <width>1280</width>
+          <height>1024</height>
           <format>R8G8B8</format>
         </image>
@@ -583,5 +585,5 @@
       <plugin name="camera_F2_controller" filename="libgazebo_ros_camera.so">
         <alwaysOn>true</alwaysOn>
-        <updateRate>30.0</updateRate>
+        <updateRate>15.0</updateRate>
         <cameraName>sensors/camera/f2</cameraName>
         <imageTopicName>image_raw</imageTopicName>

File: urdf/ig_handle_sensors.urdf.xacro (robot description, xacro)
@@ -20,4 +20,5 @@
   <!-- Lidar H (Horizontal) -->
   <!-- User: (0, -91, -268.3)mm -> ROS: (0, 0.091, 0.2683)m -->
+  <!-- Velodyne VLP-16 model: 16 channels, 360 degree sweep, 10 Hz at 600 RPM. -->
   <!-- ====================================================================== -->
   <!-- Mount pole for Lidar H -->
@@ -60,5 +61,5 @@
         <scan>
           <horizontal>
-            <samples>360</samples>
+            <samples>1800</samples>
             <resolution>1</resolution>
             <min_angle>-3.14159</min_angle>
@@ -74,5 +75,5 @@
         <range>
           <min>0.3</min>
-          <max>100.0</max>
+          <max>200.0</max>
           <resolution>0.01</resolution>
         </range>
@@ -87,5 +88,5 @@
         <frameName>lidar_h_link</frameName>
         <min_range>0.1</min_range>
-        <max_range>100.0</max_range>
+        <max_range>200.0</max_range>
         <gaussianNoise>0.005</gaussianNoise>
         <organize_cloud>false</organize_cloud>
@@ -97,4 +98,5 @@
   <!-- Lidar V (Vertical) -->
   <!-- User: (180, -126, -181)mm -> ROS: (0.180, 0.126, 0.181)m -->
+  <!-- Same VLP-16 model as lidar_h, mounted with a 90 degree pitch. -->
   <!-- ====================================================================== -->
   <!-- Mount pole for Lidar V -->
@@ -138,5 +140,5 @@
         <scan>
           <horizontal>
-            <samples>360</samples>
+            <samples>1800</samples>
             <resolution>1</resolution>
             <min_angle>-3.14159</min_angle>
@@ -152,5 +154,5 @@
         <range>
           <min>0.3</min>
-          <max>100.0</max>
+          <max>200.0</max>
           <resolution>0.01</resolution>
         </range>
@@ -165,5 +167,5 @@
         <frameName>lidar_v_link</frameName>
         <min_range>0.1</min_range>
-        <max_range>100.0</max_range>
+        <max_range>200.0</max_range>
         <gaussianNoise>0.005</gaussianNoise>
         <organize_cloud>false</organize_cloud>
@@ -174,5 +176,9 @@
   <!-- ====================================================================== -->
   <!-- Sonar -->
-  <!-- User: (0, 0, 80)mm -> ROS: (0, 0, -0.08)m (below waterline) -->
+  <!-- Imagenex DT100 profile model. User: (0, 0, 80)mm -> ROS: (0, 0, -0.08)m. -->
+  <!-- The acoustic +X axis is pitched down into ROS -Z. The ray fan models the -->
+  <!-- 480-beam, 120 degree cross-track profile. The physical 3 degree along-track -->
+  <!-- beam width is a footprint property, not extra profile beams, so Gazebo emits -->
+  <!-- one profile slice per ping. -->
   <!-- ====================================================================== -->
   <link name="sonar_link">
@@ -189,28 +195,28 @@
     <parent link="base_link"/>
     <child link="sonar_link"/>
-    <origin xyz="0 0 -0.08" rpy="0 0 0"/>
+    <origin xyz="0 0 -0.08" rpy="0 1.5708 0"/>
   </joint>
   <gazebo reference="sonar_link">
     <sensor type="ray" name="sonar">
-      <update_rate>10</update_rate>
+      <update_rate>20</update_rate>
       <ray>
          <scan>
             <horizontal>
-               <samples>64</samples>
+               <samples>480</samples>
                <resolution>1</resolution>
-               <min_angle>-0.523599</min_angle>
-               <max_angle>0.523599</max_angle>
+               <min_angle>-1.047198</min_angle>
+               <max_angle>1.047198</max_angle>
             </horizontal>
             <vertical>
-               <samples>12</samples>
+               <samples>1</samples>
                <resolution>1</resolution>
-               <min_angle>-0.174533</min_angle>
-               <max_angle>0.174533</max_angle>
+               <min_angle>0.0</min_angle>
+               <max_angle>0.0</max_angle>
             </vertical>
          </scan>
          <range>
-            <min>0.2</min>
-            <max>50.0</max>
-            <resolution>0.01</resolution>
+            <min>0.5</min>
+            <max>100.0</max>
+            <resolution>0.02</resolution>
          </range>
       </ray>
@@ -218,6 +224,6 @@
         <topicName>/sensors/sonar/scan</topicName>
         <frameName>sonar_link</frameName>
-        <min_range>0.2</min_range>
-        <max_range>50.0</max_range>
+        <min_range>0.5</min_range>
+        <max_range>100.0</max_range>
         <gaussianNoise>0.003</gaussianNoise>
         <organize_cloud>false</organize_cloud>
