Commit message: Align simulated Forge camera defaults
Co-authored-by: Aaron John Sabu <aaronjs@g.ucla.edu>

File: urdf/heron_sim.urdf.xacro (robot description, xacro)
@@ -8,6 +8,8 @@
   - lidar_v: (180, -126, -181) -> (0.180, -0.126, 0.181)
   - IMU: (65.6, -91, -203) -> (0.0656, -0.091, 0.203)
-  - Camera F1: (16.4, 21.3, -230) -> (0.0164, 0.0213, 0.230)
-  - Camera F2: (16.4, -203.3, -230) -> (0.0164, -0.2033, 0.230)
+  - Camera F1: (16.4, -21.3, -230) -> (0.0164, 0.0213, 0.230)
+  - Camera F2: (16.4, -203.3, -230) -> (0.0164, 0.2033, 0.230)
+  - Camera F3: (16.4, -21.3, -230) -> (0.0164, 0.0213, 0.230), upward
+  - Camera F4: (16.4, -203.3, -230) -> (0.0164, 0.2033, 0.230), upward
 -->
 <robot name="heron_sim" xmlns:xacro="http://www.ros.org/wiki/xacro">
@@ -261,8 +263,8 @@
   </joint>
   <!-- ====================================================================== -->
-  <!-- Camera F1 (Fisheye 1) -->
+  <!-- Camera F1 (forward left-side) -->
   <!-- User: (16.4, -21.3, -230)mm -> ROS: (0.0164, +0.0213, 0.230)m -->
   <!-- ====================================================================== -->
-  <link name="camera_F1_link">
+  <link name="F1">
     <visual>
       <geometry>
@@ -281,21 +283,91 @@
     </inertial>
   </link>
-  <joint name="camera_F1_joint" type="fixed">
-    <parent link="base_link"/>
-    <child link="camera_F1_link"/>
+  <joint name="F1_joint" type="fixed">
+    <parent link="base_link"/>
+    <child link="F1"/>
     <origin xyz="0.0164 0.0213 0.230" rpy="0 0 0"/>
   </joint>
   <!-- Camera F1 optical frame -->
-  <link name="camera_F1_optical_link"/>
-  <joint name="camera_F1_optical_joint" type="fixed">
-    <parent link="camera_F1_link"/>
-    <child link="camera_F1_optical_link"/>
+  <link name="F1_optical"/>
+  <joint name="F1_optical_joint" type="fixed">
+    <parent link="F1"/>
+    <child link="F1_optical"/>
     <origin xyz="0 0 0" rpy="-1.5708 0 -1.5708"/>
   </joint>
-  <!-- ====================================================================== -->
-  <!-- Camera F2 (Fisheye 2) -->
+  <xacro:if value="$(optenv HERON_CAMERA_F2 0)">
+    <!-- ====================================================================== -->
+    <!-- Camera F2 (forward center-ish) -->
+    <!-- User: (16.4, -203.3, -230)mm -> ROS: (0.0164, +0.2033, 0.230)m -->
+    <!-- ====================================================================== -->
+    <link name="F2">
+      <visual>
+        <geometry>
+          <box size="0.06 0.06 0.04"/>
+        </geometry>
+        <material name="sensor_blue"/>
+      </visual>
+      <collision>
+        <geometry>
+          <box size="0.06 0.06 0.04"/>
+        </geometry>
+      </collision>
+      <inertial>
+        <mass value="0.1"/>
+        <inertia ixx="0.001" ixy="0" ixz="0" iyy="0.001" iyz="0" izz="0.001"/>
+      </inertial>
+    </link>
+    <joint name="F2_joint" type="fixed">
+      <parent link="base_link"/>
+      <child link="F2"/>
+      <origin xyz="0.0164 0.2033 0.230" rpy="0 0 0"/>
+    </joint>
+    <!-- Camera F2 optical frame -->
+    <link name="F2_optical"/>
+    <joint name="F2_optical_joint" type="fixed">
+      <parent link="F2"/>
+      <child link="F2_optical"/>
+      <origin xyz="0 0 0" rpy="-1.5708 0 -1.5708"/>
+    </joint>
+  </xacro:if>
+  <xacro:if value="$(optenv HERON_CAMERA_F3 0)">
+    <!-- ====================================================================== -->
+    <!-- Camera F3 (upward left-side) -->
+    <!-- User: (16.4, -21.3, -230)mm -> ROS: (0.0164, +0.0213, 0.230)m -->
+    <!-- ====================================================================== -->
+    <link name="F3">
+      <visual>
+        <geometry>
+          <box size="0.06 0.06 0.04"/>
+        </geometry>
+        <material name="sensor_blue"/>
+      </visual>
+      <collision>
+        <geometry>
+          <box size="0.06 0.06 0.04"/>
+        </geometry>
+      </collision>
+      <inertial>
+        <mass value="0.1"/>
+        <inertia ixx="0.001" ixy="0" ixz="0" iyy="0.001" iyz="0" izz="0.001"/>
+      </inertial>
+    </link>
+    <joint name="F3_joint" type="fixed">
+      <parent link="base_link"/>
+      <child link="F3"/>
+      <origin xyz="0.0164 0.0213 0.230" rpy="0 -1.5708 0"/>
+    </joint>
+    <!-- Camera F3 optical frame -->
+    <link name="F3_optical"/>
+    <joint name="F3_optical_joint" type="fixed">
+      <parent link="F3"/>
+      <child link="F3_optical"/>
+      <origin xyz="0 0 0" rpy="-1.5708 0 -1.5708"/>
+    </joint>
+  </xacro:if>
+  <!-- ====================================================================== -->
+  <!-- Camera F4 (upward center-ish) -->
   <!-- User: (16.4, -203.3, -230)mm -> ROS: (0.0164, +0.2033, 0.230)m -->
   <!-- ====================================================================== -->
-  <link name="camera_F2_link">
+  <link name="F4">
     <visual>
       <geometry>
@@ -314,14 +386,14 @@
     </inertial>
   </link>
-  <joint name="camera_F2_joint" type="fixed">
-    <parent link="base_link"/>
-    <child link="camera_F2_link"/>
-    <origin xyz="0.0164 0.2033 0.230" rpy="0 0 0"/>
-  </joint>
-  <!-- Camera F2 optical frame -->
-  <link name="camera_F2_optical_link"/>
-  <joint name="camera_F2_optical_joint" type="fixed">
-    <parent link="camera_F2_link"/>
-    <child link="camera_F2_optical_link"/>
+  <joint name="F4_joint" type="fixed">
+    <parent link="base_link"/>
+    <child link="F4"/>
+    <origin xyz="0.0164 0.2033 0.230" rpy="0 -1.5708 0"/>
+  </joint>
+  <!-- Camera F4 optical frame -->
+  <link name="F4_optical"/>
+  <joint name="F4_optical_joint" type="fixed">
+    <parent link="F4"/>
+    <child link="F4_optical"/>
     <origin xyz="0 0 0" rpy="-1.5708 0 -1.5708"/>
   </joint>
@@ -528,5 +600,5 @@
   <!-- Camera F1 Gazebo Plugin -->
   <!-- ====================================================================== -->
-  <gazebo reference="camera_F1_link">
+  <gazebo reference="F1">
     <sensor type="camera" name="camera_F1">
       <update_rate>15.0</update_rate>
@@ -555,15 +627,87 @@
         <imageTopicName>image_raw</imageTopicName>
         <cameraInfoTopicName>camera_info</cameraInfoTopicName>
-        <frameName>camera_F1_optical_link</frameName>
+        <frameName>F1_optical</frameName>
       </plugin>
     </sensor>
   </gazebo>
-  <!-- ====================================================================== -->
-  <!-- Camera F2 Gazebo Plugin -->
-  <!-- ====================================================================== -->
-  <gazebo reference="camera_F2_link">
-    <sensor type="camera" name="camera_F2">
+  <xacro:if value="$(optenv HERON_CAMERA_F2 0)">
+    <!-- ====================================================================== -->
+    <!-- Camera F2 Gazebo Plugin -->
+    <!-- ====================================================================== -->
+    <gazebo reference="F2">
+      <sensor type="camera" name="camera_F2">
+        <update_rate>15.0</update_rate>
+        <camera name="F2">
+          <horizontal_fov>1.60</horizontal_fov>
+          <image>
+            <width>1280</width>
+            <height>1024</height>
+            <format>R8G8B8</format>
+          </image>
+          <clip>
+            <near>0.02</near>
+            <far>100</far>
+          </clip>
+          <visibility_mask>4294967294</visibility_mask>
+          <noise>
+            <type>gaussian</type>
+            <mean>0.0</mean>
+            <stddev>0.007</stddev>
+          </noise>
+        </camera>
+        <plugin name="camera_F2_controller" filename="libgazebo_ros_camera.so">
+          <alwaysOn>true</alwaysOn>
+          <updateRate>15.0</updateRate>
+          <cameraName>sensors/camera/f2</cameraName>
+          <imageTopicName>image_raw</imageTopicName>
+          <cameraInfoTopicName>camera_info</cameraInfoTopicName>
+          <frameName>F2_optical</frameName>
+        </plugin>
+      </sensor>
+    </gazebo>
+  </xacro:if>
+  <xacro:if value="$(optenv HERON_CAMERA_F3 0)">
+    <!-- ====================================================================== -->
+    <!-- Camera F3 Gazebo Plugin -->
+    <!-- ====================================================================== -->
+    <gazebo reference="F3">
+      <sensor type="camera" name="camera_F3">
+        <update_rate>15.0</update_rate>
+        <camera name="F3">
+          <horizontal_fov>1.60</horizontal_fov>
+          <image>
+            <width>1280</width>
+            <height>1024</height>
+            <format>R8G8B8</format>
+          </image>
+          <clip>
+            <near>0.02</near>
+            <far>100</far>
+          </clip>
+          <visibility_mask>4294967294</visibility_mask>
+          <noise>
+            <type>gaussian</type>
+            <mean>0.0</mean>
+            <stddev>0.007</stddev>
+          </noise>
+        </camera>
+        <plugin name="camera_F3_controller" filename="libgazebo_ros_camera.so">
+          <alwaysOn>true</alwaysOn>
+          <updateRate>15.0</updateRate>
+          <cameraName>sensors/camera/f3</cameraName>
+          <imageTopicName>image_raw</imageTopicName>
+          <cameraInfoTopicName>camera_info</cameraInfoTopicName>
+          <frameName>F3_optical</frameName>
+        </plugin>
+      </sensor>
+    </gazebo>
+  </xacro:if>
+  <!-- ====================================================================== -->
+  <!-- Camera F4 Gazebo Plugin -->
+  <!-- ====================================================================== -->
+  <gazebo reference="F4">
+    <sensor type="camera" name="camera_F4">
       <update_rate>15.0</update_rate>
-      <camera name="F2">
+      <camera name="F4">
         <horizontal_fov>1.60</horizontal_fov>
         <image>
@@ -583,11 +727,11 @@
         </noise>
       </camera>
-      <plugin name="camera_F2_controller" filename="libgazebo_ros_camera.so">
+      <plugin name="camera_F4_controller" filename="libgazebo_ros_camera.so">
         <alwaysOn>true</alwaysOn>
         <updateRate>15.0</updateRate>
-        <cameraName>sensors/camera/f2</cameraName>
+        <cameraName>sensors/camera/f4</cameraName>
         <imageTopicName>image_raw</imageTopicName>
         <cameraInfoTopicName>camera_info</cameraInfoTopicName>
-        <frameName>camera_F2_optical_link</frameName>
+        <frameName>F4_optical</frameName>
       </plugin>
     </sensor>

File: urdf/ig_handle_sensors.urdf.xacro (robot description, xacro)
@@ -250,128 +250,111 @@
     <origin xyz="0.0164 0.1 0.13" rpy="0 0 0"/>
   </joint>
-  <!-- ====================================================================== -->
-  <!-- Camera F1 (Fisheye 1) -->
-  <!-- User: (16.4, -21.3, -230)mm -> ROS: (0.0164, 0.0213, 0.230)m -->
-  <!-- ====================================================================== -->
-  <link name="camera_F1_link">
-    <visual>
-      <geometry><box size="0.06 0.06 0.04"/></geometry>
-      <material name="sensor_blue"/>
-    </visual>
-    <inertial>
-      <mass value="0.1"/>
-      <inertia ixx="0.001" ixy="0" ixz="0" iyy="0.001" iyz="0" izz="0.001"/>
-    </inertial>
-  </link>
-  <joint name="camera_F1_joint" type="fixed">
-    <parent link="base_link"/>
-    <child link="camera_F1_link"/>
-    <origin xyz="0.0164 0.0213 0.230" rpy="0 0 0"/>
-  </joint>
-  <link name="camera_F1_optical_link"/>
-  <joint name="camera_F1_optical_joint" type="fixed">
-    <parent link="camera_F1_link"/>
-    <child link="camera_F1_optical_link"/>
-    <origin xyz="0 0 0" rpy="-1.5708 0 -1.5708"/>
-  </joint>
-  <gazebo reference="camera_F1_link">
-    <sensor type="camera" name="camera_F1_sensor">
-      <update_rate>15.0</update_rate>
-      <camera name="front_camera">
-        <horizontal_fov>1.60</horizontal_fov>
-        <image>
-          <width>1280</width>
-          <height>1024</height>
-          <format>R8G8B8</format>
-        </image>
-        <clip>
-          <near>0.02</near>
-          <far>100</far>
-        </clip>
-        <visibility_mask>4294967294</visibility_mask>
-        <noise>
-          <type>gaussian</type>
-          <mean>0.0</mean>
-          <stddev>0.007</stddev>
-        </noise>
-      </camera>
-      <plugin name="camera_controller" filename="libgazebo_ros_camera.so">
-        <alwaysOn>true</alwaysOn>
-        <updateRate>15.0</updateRate>
-        <cameraName>sensors/camera/f1</cameraName>
-        <imageTopicName>image_raw</imageTopicName>
-        <cameraInfoTopicName>camera_info</cameraInfoTopicName>
-        <frameName>camera_F1_optical_link</frameName>
-        <hackBaseline>0.07</hackBaseline>
-        <distortionK1>-0.0100</distortionK1>
-        <distortionK2>0.0030</distortionK2>
-        <distortionK3>-0.0020</distortionK3>
-        <distortionT1>0.0</distortionT1>
-        <distortionT2>0.0</distortionT2>
-      </plugin>
-    </sensor>
-  </gazebo>
-  <!-- ====================================================================== -->
-  <!-- Camera F2 (Fisheye 2) -->
-  <!-- User: (16.4, -203.3, -230)mm -> ROS: (0.0164, 0.2033, 0.230)m -->
-  <!-- ====================================================================== -->
-  <link name="camera_F2_link">
-    <visual>
-      <geometry><box size="0.06 0.06 0.04"/></geometry>
-      <material name="sensor_blue"/>
-    </visual>
-    <inertial>
-      <mass value="0.1"/>
-      <inertia ixx="0.001" ixy="0" ixz="0" iyy="0.001" iyz="0" izz="0.001"/>
-    </inertial>
-  </link>
-  <joint name="camera_F2_joint" type="fixed">
-    <parent link="base_link"/>
-    <child link="camera_F2_link"/>
-    <origin xyz="0.0164 0.2033 0.230" rpy="0 0 0"/>
-  </joint>
-  <link name="camera_F2_optical_link"/>
-  <joint name="camera_F2_optical_joint" type="fixed">
-    <parent link="camera_F2_link"/>
-    <child link="camera_F2_optical_link"/>
-    <origin xyz="0 0 0" rpy="-1.5708 0 -1.5708"/>
-  </joint>
-  <gazebo reference="camera_F2_link">
-    <sensor type="camera" name="camera_F2_sensor">
-      <update_rate>15.0</update_rate>
-      <camera name="front_camera_right">
-        <horizontal_fov>1.60</horizontal_fov>
-        <image>
-          <width>1280</width>
-          <height>1024</height>
-          <format>R8G8B8</format>
-        </image>
-        <clip>
-          <near>0.02</near>
-          <far>100</far>
-        </clip>
-        <visibility_mask>4294967294</visibility_mask>
-        <noise>
-          <type>gaussian</type>
-          <mean>0.0</mean>
-          <stddev>0.007</stddev>
-        </noise>
-      </camera>
-      <plugin name="camera_F2_controller" filename="libgazebo_ros_camera.so">
-        <alwaysOn>true</alwaysOn>
-        <updateRate>15.0</updateRate>
-        <cameraName>sensors/camera/f2</cameraName>
-        <imageTopicName>image_raw</imageTopicName>
-        <cameraInfoTopicName>camera_info</cameraInfoTopicName>
-        <frameName>camera_F2_optical_link</frameName>
-        <hackBaseline>0.07</hackBaseline>
-        <distortionK1>-0.0090</distortionK1>
-        <distortionK2>0.0028</distortionK2>
-        <distortionK3>-0.0019</distortionK3>
-        <distortionT1>0.0</distortionT1>
-        <distortionT2>0.0</distortionT2>
-      </plugin>
-    </sensor>
-  </gazebo>
+  <xacro:macro name="ig_handle_forge_camera"
+               params="id xyz rpy topic_suffix camera_name distortion_k1 distortion_k2 distortion_k3">
+    <link name="${id}">
+      <visual>
+        <geometry><box size="0.06 0.06 0.04"/></geometry>
+        <material name="sensor_blue"/>
+      </visual>
+      <inertial>
+        <mass value="0.1"/>
+        <inertia ixx="0.001" ixy="0" ixz="0" iyy="0.001" iyz="0" izz="0.001"/>
+      </inertial>
+    </link>
+    <joint name="${id}_joint" type="fixed">
+      <parent link="base_link"/>
+      <child link="${id}"/>
+      <origin xyz="${xyz}" rpy="${rpy}"/>
+    </joint>
+    <link name="${id}_optical"/>
+    <joint name="${id}_optical_joint" type="fixed">
+      <parent link="${id}"/>
+      <child link="${id}_optical"/>
+      <origin xyz="0 0 0" rpy="-1.5708 0 -1.5708"/>
+    </joint>
+    <gazebo reference="${id}">
+      <sensor type="camera" name="camera_${id}_sensor">
+        <update_rate>15.0</update_rate>
+        <camera name="${camera_name}">
+          <horizontal_fov>1.60</horizontal_fov>
+          <image>
+            <width>1280</width>
+            <height>1024</height>
+            <format>R8G8B8</format>
+          </image>
+          <clip>
+            <near>0.02</near>
+            <far>100</far>
+          </clip>
+          <visibility_mask>4294967294</visibility_mask>
+          <noise>
+            <type>gaussian</type>
+            <mean>0.0</mean>
+            <stddev>0.007</stddev>
+          </noise>
+        </camera>
+        <plugin name="camera_${id}_controller" filename="libgazebo_ros_camera.so">
+          <alwaysOn>true</alwaysOn>
+          <updateRate>15.0</updateRate>
+          <cameraName>sensors/camera/${topic_suffix}</cameraName>
+          <imageTopicName>image_raw</imageTopicName>
+          <cameraInfoTopicName>camera_info</cameraInfoTopicName>
+          <frameName>${id}_optical</frameName>
+          <hackBaseline>0.07</hackBaseline>
+          <distortionK1>${distortion_k1}</distortionK1>
+          <distortionK2>${distortion_k2}</distortionK2>
+          <distortionK3>${distortion_k3}</distortionK3>
+          <distortionT1>0.0</distortionT1>
+          <distortionT2>0.0</distortionT2>
+        </plugin>
+      </sensor>
+    </gazebo>
+  </xacro:macro>
+  <!-- ====================================================================== -->
+  <!-- Forge camera stack -->
+  <!-- F1/F2 face forward; F3/F4 face upward. F1/F3 are left-side mounts, and
+       F2/F4 are center-ish mounts. These frame names intentionally match the
+       real Forge driver frame IDs and shared sensor YAML. -->
+  <!-- ====================================================================== -->
+  <xacro:if value="$(optenv HERON_CAMERA_F1 1)">
+    <xacro:ig_handle_forge_camera id="F1"
+                                  xyz="0.0164 0.0213 0.230"
+                                  rpy="0 0 0"
+                                  topic_suffix="f1"
+                                  camera_name="forward_left"
+                                  distortion_k1="-0.0100"
+                                  distortion_k2="0.0030"
+                                  distortion_k3="-0.0020"/>
+  </xacro:if>
+  <xacro:if value="$(optenv HERON_CAMERA_F2 0)">
+    <xacro:ig_handle_forge_camera id="F2"
+                                  xyz="0.0164 0.2033 0.230"
+                                  rpy="0 0 0"
+                                  topic_suffix="f2"
+                                  camera_name="forward_center"
+                                  distortion_k1="-0.0090"
+                                  distortion_k2="0.0028"
+                                  distortion_k3="-0.0019"/>
+  </xacro:if>
+  <xacro:if value="$(optenv HERON_CAMERA_F3 0)">
+    <xacro:ig_handle_forge_camera id="F3"
+                                  xyz="0.0164 0.0213 0.230"
+                                  rpy="0 -1.5708 0"
+                                  topic_suffix="f3"
+                                  camera_name="upward_left"
+                                  distortion_k1="-0.0100"
+                                  distortion_k2="0.0030"
+                                  distortion_k3="-0.0020"/>
+  </xacro:if>
+  <xacro:if value="$(optenv HERON_CAMERA_F4 1)">
+    <xacro:ig_handle_forge_camera id="F4"
+                                  xyz="0.0164 0.2033 0.230"
+                                  rpy="0 -1.5708 0"
+                                  topic_suffix="f4"
+                                  camera_name="upward_center"
+                                  distortion_k1="-0.0090"
+                                  distortion_k2="0.0028"
+                                  distortion_k3="-0.0019"/>
+  </xacro:if>
   <!-- ====================================================================== -->
   <!-- IMU Visual (for debugging) -->

Commit message: Correct horizontal VLP16 center offset

File: urdf/heron_sim.urdf.xacro (robot description, xacro)
@@ -5,5 +5,7 @@
   Physical sensor positions (mm, z-down) converted to URDF (meters, z-up):
   - Water level: z = -40mm -> boat floats at z=-0.04m
-  - lidar_h: (0, -91, -268.3) -> (0, -0.091, 0.2683)
+  - lidar_h measured cable-side/top reference: (0, -91, -268.3)
+    VLP-16 center origin after +50.86mm away from cable and -36.19mm from top:
+    (0, -141.86, -232.11) -> (0, +0.14186, 0.23211)
   - lidar_v: (180, -126, -181) -> (0.180, -0.126, 0.181)
   - IMU: (65.6, -91, -203) -> (0.0656, -0.091, 0.203)
@@ -150,5 +152,8 @@
   <!-- ====================================================================== -->
   <!-- Horizontal Lidar (lidar_h) -->
-  <!-- User: (0, -91, -268.3)mm -> ROS: (0, +0.091, 0.2683)m -->
+  <!-- User measured cable-side/top reference: (0, -91, -268.3)mm.
+       VLP-16 origin is sensor center: cable is on -Y_lidar, body is
+       101.72 mm diameter x 72.38 mm tall.
+       Corrected center -> ROS: (0, +0.14186, 0.23211)m. -->
   <!-- ====================================================================== -->
   <!-- Lidar H mount pole -->
@@ -174,5 +179,5 @@
     <visual>
       <geometry>
-        <cylinder radius="0.05" length="0.07"/>
+        <cylinder radius="0.05086" length="0.07238"/>
       </geometry>
       <origin xyz="0 0 0" rpy="0 0 0"/>
@@ -181,5 +186,5 @@
     <collision>
       <geometry>
-        <cylinder radius="0.05" length="0.07"/>
+        <cylinder radius="0.05086" length="0.07238"/>
       </geometry>
     </collision>
@@ -192,5 +197,5 @@
     <parent link="base_link"/>
     <child link="lidar_h_link"/>
-    <origin xyz="0 0.091 0.2683" rpy="0 0 0"/>
+    <origin xyz="0 0.14186 0.23211" rpy="0 0 0"/>
   </joint>
   <!-- ====================================================================== -->

File: urdf/ig_handle_sensors.urdf.xacro (robot description, xacro)
@@ -19,5 +19,8 @@
   <!-- ====================================================================== -->
   <!-- Lidar H (Horizontal) -->
-  <!-- User: (0, -91, -268.3)mm -> ROS: (0, 0.091, 0.2683)m -->
+  <!-- User measured cable-side/top reference: (0, -91, -268.3)mm.
+       VLP-16 origin is sensor center: cable is on -Y_lidar, body is
+       101.72 mm diameter x 72.38 mm tall.
+       Corrected center -> ROS: (0, 0.14186, 0.23211)m. -->
   <!-- Velodyne VLP-16 model: 16 channels, 360 degree sweep, 10 Hz at 600 RPM. -->
   <!-- ====================================================================== -->
@@ -40,5 +43,5 @@
   <link name="lidar_h_link">
     <visual>
-      <geometry><cylinder radius="0.05" length="0.07"/></geometry>
+      <geometry><cylinder radius="0.05086" length="0.07238"/></geometry>
       <material name="sensor_black"/>
     </visual>
@@ -51,5 +54,5 @@
     <parent link="base_link"/>
     <child link="lidar_h_link"/>
-    <origin xyz="0 0.091 0.2683" rpy="0 0 0"/>
+    <origin xyz="0 0.14186 0.23211" rpy="0 0 0"/>
   </joint>
   <gazebo reference="lidar_h_link">
