Commit message: Align Heron sensor frames with cable-aft mounts

File: urdf/heron_sim.urdf.xacro (robot description, xacro)
@@ -5,7 +5,9 @@
   Physical sensor positions (mm, z-down) converted to URDF (meters, z-up):
   - Water level: z = -40mm -> boat floats at z=-0.04m
-  - lidar_h measured cable-side/top reference: (0, -91, -268.3)
-    VLP-16 center origin after +50.86mm away from cable and -36.19mm from top:
-    (0, -141.86, -232.11) -> (0, +0.14186, 0.23211)
+  - lidar_h VLP-16 cable is on -Y_lidar and exits stern, so lidar_h is yawed
+    -90 deg. Relative to the current IMU cable/reference point, the lidar cable
+    is 3.72mm forward, 7.15mm left, and 35.64mm higher; the VLP center is
+    another 50.86mm forward and 36.19mm lower:
+    (120.18, -98.15, -202.45) -> (0.12018, +0.09815, 0.20245)
   - lidar_v: (180, -126, -181) -> (0.180, -0.126, 0.181)
   - IMU: (65.6, -91, -203) -> (0.0656, -0.091, 0.203)
@@ -102,6 +104,7 @@
   <!-- ====================================================================== -->
   <!-- IMU Sensor -->
-  <!-- User: (65.6, -91, -203)mm -> ROS: (0.0656, +0.091, 0.203)m -->
-  <!-- Y negated: user y-right, ROS y-left -->
+  <!-- User: (65.6, -91, -203)mm -> ROS: (0.0656, +0.091, 0.203)m.
+       Xsens cable exits stern and label side faces down, so imu_link is
+       pitched 180 deg relative to base_link. -->
   <!-- ====================================================================== -->
   <link name="imu_link">
@@ -120,5 +123,5 @@
     <parent link="base_link"/>
     <child link="imu_link"/>
-    <origin xyz="0.0656 0.091 0.203" rpy="0 0 0"/>
+    <origin xyz="0.0656 0.091 0.203" rpy="0 3.141592653589793 0"/>
   </joint>
   <gazebo>
@@ -152,8 +155,10 @@
   <!-- ====================================================================== -->
   <!-- Horizontal Lidar (lidar_h) -->
-  <!-- User measured cable-side/top reference: (0, -91, -268.3)mm.
-       VLP-16 origin is sensor center: cable is on -Y_lidar, body is
-       101.72 mm diameter x 72.38 mm tall.
-       Corrected center -> ROS: (0, +0.14186, 0.23211)m. -->
+  <!-- VLP-16 origin is sensor center. The cable is on -Y_lidar and exits
+       toward the stern, so the sensor frame is yawed -90 deg relative to the
+       boat. Relative to the current IMU cable/reference point, the lidar cable
+       is 3.72 mm forward, 7.15 mm left, and 35.64 mm higher; the VLP center is
+       another 50.86 mm forward and 36.19 mm lower.
+       Corrected center -> ROS: (0.12018, +0.09815, 0.20245)m. -->
   <!-- ====================================================================== -->
   <!-- Lidar H mount pole -->
@@ -174,5 +179,5 @@
     <parent link="base_link"/>
     <child link="lidar_h_mount"/>
-    <origin xyz="0 0.091 0.16" rpy="0 0 0"/>
+    <origin xyz="0.12018 0.09815 0.16" rpy="0 0 0"/>
   </joint>
   <link name="lidar_h_link">
@@ -197,5 +202,5 @@
     <parent link="base_link"/>
     <child link="lidar_h_link"/>
-    <origin xyz="0 0.14186 0.23211" rpy="0 0 0"/>
+    <origin xyz="0.12018 0.09815 0.20245" rpy="0 0 -1.5707963267948966"/>
   </joint>
   <!-- ====================================================================== -->

File: urdf/ig_handle_sensors.urdf.xacro (robot description, xacro)
@@ -19,8 +19,10 @@
   <!-- ====================================================================== -->
   <!-- Lidar H (Horizontal) -->
-  <!-- User measured cable-side/top reference: (0, -91, -268.3)mm.
-       VLP-16 origin is sensor center: cable is on -Y_lidar, body is
-       101.72 mm diameter x 72.38 mm tall.
-       Corrected center -> ROS: (0, 0.14186, 0.23211)m. -->
+  <!-- VLP-16 origin is sensor center. The cable is on -Y_lidar and exits
+       toward the stern, so the sensor frame is yawed -90 deg relative to the
+       boat. Relative to the current IMU cable/reference point, the lidar cable
+       is 3.72 mm forward, 7.15 mm left, and 35.64 mm higher; the VLP center is
+       another 50.86 mm forward and 36.19 mm lower.
+       Corrected center -> ROS: (0.12018, 0.09815, 0.20245)m. -->
   <!-- Velodyne VLP-16 model: 16 channels, 360 degree sweep, 10 Hz at 600 RPM. -->
   <!-- ====================================================================== -->
@@ -39,5 +41,5 @@
     <parent link="base_link"/>
     <child link="lidar_h_mount"/>
-    <origin xyz="0 0.091 0.16" rpy="0 0 0"/>
+    <origin xyz="0.12018 0.09815 0.16" rpy="0 0 0"/>
   </joint>
   <link name="lidar_h_link">
@@ -54,5 +56,5 @@
     <parent link="base_link"/>
     <child link="lidar_h_link"/>
-    <origin xyz="0 0.14186 0.23211" rpy="0 0 0"/>
+    <origin xyz="0.12018 0.09815 0.20245" rpy="0 0 -1.5707963267948966"/>
   </joint>
   <gazebo reference="lidar_h_link">
@@ -362,5 +364,7 @@
   <!-- ====================================================================== -->
   <!-- IMU Visual (for debugging) -->
-  <!-- User: (65.6, -91, -203)mm -> ROS: (0.0656, 0.091, 0.203)m -->
+  <!-- User: (65.6, -91, -203)mm -> ROS: (0.0656, 0.091, 0.203)m.
+       Xsens cable exits stern and label side faces down, so imu_link is
+       pitched 180 deg relative to base_link. -->
   <!-- Note: imu_link is already defined in base Heron URDF, just add visual -->
   <!-- ====================================================================== -->
@@ -379,5 +383,5 @@
     <parent link="base_link"/>
     <child link="debug_extra_link"/>
-    <origin xyz="0.0656 0.091 0.203" rpy="0 0 0"/>
+    <origin xyz="0.0656 0.091 0.203" rpy="0 3.141592653589793 0"/>
   </joint>
   <gazebo>

Commit message: Correct Heron VLP16 cable height in URDF

File: urdf/heron_sim.urdf.xacro (robot description, xacro)
@@ -8,6 +8,6 @@
     -90 deg. Relative to the current IMU cable/reference point, the lidar cable
     is 3.72mm forward, 7.15mm left, and 35.64mm higher; the VLP center is
-    another 50.86mm forward and 36.19mm lower:
-    (120.18, -98.15, -202.45) -> (0.12018, +0.09815, 0.20245)
+    another 50.86mm forward from the cable side and 36.19mm above the cable
+    exit: (120.18, -98.15, -274.83) -> (0.12018, +0.09815, 0.27483)
   - lidar_v: (180, -126, -181) -> (0.180, -0.126, 0.181)
   - IMU: (65.6, -91, -203) -> (0.0656, -0.091, 0.203)
@@ -159,6 +159,6 @@
        boat. Relative to the current IMU cable/reference point, the lidar cable
        is 3.72 mm forward, 7.15 mm left, and 35.64 mm higher; the VLP center is
-       another 50.86 mm forward and 36.19 mm lower.
-       Corrected center -> ROS: (0.12018, +0.09815, 0.20245)m. -->
+       another 50.86 mm forward from the cable side and 36.19 mm above the cable
+       exit. Corrected center -> ROS: (0.12018, +0.09815, 0.27483)m. -->
   <!-- ====================================================================== -->
   <!-- Lidar H mount pole -->
@@ -202,5 +202,5 @@
     <parent link="base_link"/>
     <child link="lidar_h_link"/>
-    <origin xyz="0.12018 0.09815 0.20245" rpy="0 0 -1.5707963267948966"/>
+    <origin xyz="0.12018 0.09815 0.27483" rpy="0 0 -1.5707963267948966"/>
   </joint>
   <!-- ====================================================================== -->

File: urdf/ig_handle_sensors.urdf.xacro (robot description, xacro)
@@ -23,6 +23,6 @@
        boat. Relative to the current IMU cable/reference point, the lidar cable
        is 3.72 mm forward, 7.15 mm left, and 35.64 mm higher; the VLP center is
-       another 50.86 mm forward and 36.19 mm lower.
-       Corrected center -> ROS: (0.12018, 0.09815, 0.20245)m. -->
+       another 50.86 mm forward from the cable side and 36.19 mm above the cable
+       exit. Corrected center -> ROS: (0.12018, 0.09815, 0.27483)m. -->
   <!-- Velodyne VLP-16 model: 16 channels, 360 degree sweep, 10 Hz at 600 RPM. -->
   <!-- ====================================================================== -->
@@ -56,5 +56,5 @@
     <parent link="base_link"/>
     <child link="lidar_h_link"/>
-    <origin xyz="0.12018 0.09815 0.20245" rpy="0 0 -1.5707963267948966"/>
+    <origin xyz="0.12018 0.09815 0.27483" rpy="0 0 -1.5707963267948966"/>
   </joint>
   <gazebo reference="lidar_h_link">

Commit message: Align Heron sensor frames with mounts

File: urdf/heron_sim.urdf.xacro (robot description, xacro)
@@ -10,5 +10,5 @@
     another 50.86mm forward from the cable side and 36.19mm above the cable
     exit: (120.18, -98.15, -274.83) -> (0.12018, +0.09815, 0.27483)
-  - lidar_v: (180, -126, -181) -> (0.180, -0.126, 0.181)
+  - lidar_v: (180, -126, -181) -> (0.180, +0.126, 0.181)
   - IMU: (65.6, -91, -203) -> (0.0656, -0.091, 0.203)
   - Camera F1: (16.4, -21.3, -230) -> (0.0164, 0.0213, 0.230)
@@ -105,6 +105,6 @@
   <!-- IMU Sensor -->
   <!-- User: (65.6, -91, -203)mm -> ROS: (0.0656, +0.091, 0.203)m.
-       Xsens cable exits stern and label side faces down, so imu_link is
-       pitched 180 deg relative to base_link. -->
+       Xsens frame is mounted with +X forward, +Y starboard/right, and +Z down
+       toward the water. -->
   <!-- ====================================================================== -->
   <link name="imu_link">
@@ -123,5 +123,5 @@
     <parent link="base_link"/>
     <child link="imu_link"/>
-    <origin xyz="0.0656 0.091 0.203" rpy="0 3.141592653589793 0"/>
+    <origin xyz="0.0656 0.091 0.203" rpy="3.141592653589793 0 0"/>
   </joint>
   <gazebo>
@@ -207,4 +207,5 @@
   <!-- Vertical Lidar (lidar_v) -->
   <!-- User: (180, -126, -181)mm -> ROS: (0.180, +0.126, 0.181)m -->
+  <!-- Vertical VLP-16 frame: +X starboard/right, +Y up, +Z aft/stern. -->
   <!-- ====================================================================== -->
   <!-- Lidar V mount pole -->
@@ -248,6 +249,5 @@
     <parent link="base_link"/>
     <child link="lidar_v_link"/>
-    <!-- Rotated 90deg pitch to convert the VLP-16 into a vertical sweep. -->
-    <origin xyz="0.180 0.126 0.181" rpy="0 1.5708 0"/>
+    <origin xyz="0.180 0.126 0.181" rpy="1.5707963267948966 0 -1.5707963267948966"/>
   </joint>
   <!-- ====================================================================== -->
@@ -563,9 +563,9 @@
   <!-- ====================================================================== -->
   <!-- Vertical Lidar Gazebo Plugin -->
-  <!-- Same VLP-16 model as lidar_h, mounted with a 90 degree pitch. -->
+  <!-- Same VLP-16 model as lidar_h; lidar_v_link already carries the mount frame. -->
   <!-- ====================================================================== -->
   <gazebo reference="lidar_v_link">
     <sensor type="ray" name="lidar_v_sensor">
-      <pose>0 0 0 1.5708 0 0</pose>
+      <pose>0 0 0 0 0 0</pose>
       <visualize>false</visualize>
       <update_rate>10</update_rate>

File: urdf/ig_handle_sensors.urdf.xacro (robot description, xacro)
@@ -103,5 +103,5 @@
   <!-- Lidar V (Vertical) -->
   <!-- User: (180, -126, -181)mm -> ROS: (0.180, 0.126, 0.181)m -->
-  <!-- Same VLP-16 model as lidar_h, mounted with a 90 degree pitch. -->
+  <!-- Vertical VLP-16 frame: +X starboard/right, +Y up, +Z aft/stern. -->
   <!-- ====================================================================== -->
   <!-- Mount pole for Lidar V -->
@@ -134,6 +134,5 @@
     <parent link="base_link"/>
     <child link="lidar_v_link"/>
-    <!-- Rotated 90deg pitch for vertical scanning -->
-    <origin xyz="0.180 0.126 0.181" rpy="0 1.5708 0"/>
+    <origin xyz="0.180 0.126 0.181" rpy="1.5707963267948966 0 -1.5707963267948966"/>
   </joint>
   <gazebo reference="lidar_v_link">
@@ -365,6 +364,6 @@
   <!-- IMU Visual (for debugging) -->
   <!-- User: (65.6, -91, -203)mm -> ROS: (0.0656, 0.091, 0.203)m.
-       Xsens cable exits stern and label side faces down, so imu_link is
-       pitched 180 deg relative to base_link. -->
+       Xsens frame is mounted with +X forward, +Y starboard/right, and +Z down
+       toward the water. -->
   <!-- Note: imu_link is already defined in base Heron URDF, just add visual -->
   <!-- ====================================================================== -->
@@ -383,5 +382,5 @@
     <parent link="base_link"/>
     <child link="debug_extra_link"/>
-    <origin xyz="0.0656 0.091 0.203" rpy="0 3.141592653589793 0"/>
+    <origin xyz="0.0656 0.091 0.203" rpy="3.141592653589793 0 0"/>
   </joint>
   <gazebo>

Commit message: Update Heron vertical lidar mount offset

File: urdf/heron_sim.urdf.xacro (robot description, xacro)
@@ -10,5 +10,5 @@
     another 50.86mm forward from the cable side and 36.19mm above the cable
     exit: (120.18, -98.15, -274.83) -> (0.12018, +0.09815, 0.27483)
-  - lidar_v: (180, -126, -181) -> (0.180, +0.126, 0.181)
+  - lidar_v center: lidar_h center x - 0.10298m -> (0.01720, +0.126, 0.181)
   - IMU: (65.6, -91, -203) -> (0.0656, -0.091, 0.203)
   - Camera F1: (16.4, -21.3, -230) -> (0.0164, 0.0213, 0.230)
@@ -104,7 +104,8 @@
   <!-- ====================================================================== -->
   <!-- IMU Sensor -->
-  <!-- User: (65.6, -91, -203)mm -> ROS: (0.0656, +0.091, 0.203)m.
-       Xsens frame is mounted with +X forward, +Y starboard/right, and +Z down
-       toward the water. -->
+  <!-- Current connector/reference value: (0.0656, +0.091, 0.203)m.
+       Encased MTi-30 AHRS device ID 0368xxxx: connector side is -X and exits
+       aft, the unit is upside down, so +X is forward, +Y is starboard/right,
+       and +Z points down toward the water. -->
   <!-- ====================================================================== -->
   <link name="imu_link">
@@ -206,5 +207,7 @@
   <!-- ====================================================================== -->
   <!-- Vertical Lidar (lidar_v) -->
-  <!-- User: (180, -126, -181)mm -> ROS: (0.180, +0.126, 0.181)m -->
+  <!-- Vertical VLP reference plane is 0.10298 m behind the lidar_h connector.
+       With lidar_v +Z aft and the VLP origin at sensor center, the center is
+       one radius forward from that plane: (0.01720, +0.126, 0.181)m. -->
   <!-- Vertical VLP-16 frame: +X starboard/right, +Y up, +Z aft/stern. -->
   <!-- ====================================================================== -->
@@ -226,5 +229,5 @@
     <parent link="base_link"/>
     <child link="lidar_v_mount"/>
-    <origin xyz="0.180 0.126 0.11" rpy="0 0 0"/>
+    <origin xyz="0.01720 0.126 0.11" rpy="0 0 0"/>
   </joint>
   <link name="lidar_v_link">
@@ -249,5 +252,5 @@
     <parent link="base_link"/>
     <child link="lidar_v_link"/>
-    <origin xyz="0.180 0.126 0.181" rpy="1.5707963267948966 0 -1.5707963267948966"/>
+    <origin xyz="0.01720 0.126 0.181" rpy="1.5707963267948966 0 -1.5707963267948966"/>
   </joint>
   <!-- ====================================================================== -->

File: urdf/ig_handle_sensors.urdf.xacro (robot description, xacro)
@@ -102,5 +102,7 @@
   <!-- ====================================================================== -->
   <!-- Lidar V (Vertical) -->
-  <!-- User: (180, -126, -181)mm -> ROS: (0.180, 0.126, 0.181)m -->
+  <!-- Vertical VLP reference plane is 0.10298 m behind the lidar_h connector.
+       With lidar_v +Z aft and the VLP origin at sensor center, the center is
+       one radius forward from that plane: (0.01720, 0.126, 0.181)m. -->
   <!-- Vertical VLP-16 frame: +X starboard/right, +Y up, +Z aft/stern. -->
   <!-- ====================================================================== -->
@@ -119,5 +121,5 @@
     <parent link="base_link"/>
     <child link="lidar_v_mount"/>
-    <origin xyz="0.180 0.126 0.11" rpy="0 0 0"/>
+    <origin xyz="0.01720 0.126 0.11" rpy="0 0 0"/>
   </joint>
   <link name="lidar_v_link">
@@ -134,5 +136,5 @@
     <parent link="base_link"/>
     <child link="lidar_v_link"/>
-    <origin xyz="0.180 0.126 0.181" rpy="1.5707963267948966 0 -1.5707963267948966"/>
+    <origin xyz="0.01720 0.126 0.181" rpy="1.5707963267948966 0 -1.5707963267948966"/>
   </joint>
   <gazebo reference="lidar_v_link">
@@ -363,7 +365,8 @@
   <!-- ====================================================================== -->
   <!-- IMU Visual (for debugging) -->
-  <!-- User: (65.6, -91, -203)mm -> ROS: (0.0656, 0.091, 0.203)m.
-       Xsens frame is mounted with +X forward, +Y starboard/right, and +Z down
-       toward the water. -->
+  <!-- Current connector/reference value: (0.0656, 0.091, 0.203)m.
+       Encased MTi-30 AHRS device ID 0368xxxx: connector side is -X and exits
+       aft, the unit is upside down, so +X is forward, +Y is starboard/right,
+       and +Z points down toward the water. -->
   <!-- Note: imu_link is already defined in base Heron URDF, just add visual -->
   <!-- ====================================================================== -->
