Commit message: Sync simulator sensor extrinsics

File: urdf/heron_sim.urdf.xacro (robot description, xacro)
@@ -3,13 +3,9 @@
   Standalone Heron simulation URDF
   Sensor positions match physical IG-Handle boat configuration
-  Physical sensor positions (mm, z-down) converted to URDF (meters, z-up):
+  Physical sensor positions converted to URDF base_link (meters):
   - Water level: z = -40mm -> boat floats at z=-0.04m
-  - lidar_h VLP-16 cable is on -Y_lidar and exits stern, so lidar_h is yawed
-    -90 deg. Relative to the current IMU cable/reference point, the lidar cable
-    is 3.72mm forward, 7.15mm left, and 35.64mm higher; the VLP center is
-    another 50.86mm forward from the cable side and 36.19mm above the cable
-    exit: (120.18, -98.15, -274.83) -> (0.12018, +0.09815, 0.27483)
-  - lidar_v center: lidar_h center x - 0.10298m -> (0.01720, +0.126, 0.181)
-  - IMU: (65.6, -91, -203) -> (0.0656, -0.091, 0.203)
+  - lidar_h VLP-16 origin: (0.00000, +0.13000, 0.29654), yaw -90 deg
+  - lidar_v VLP-16 origin: (-0.19003, +0.12234, 0.18068), roll 90 deg + yaw -90 deg
+  - imu_link origin: (-0.01188, +0.12755, 0.23412), roll 180 deg
   - Camera F1: (16.4, -21.3, -230) -> (0.0164, 0.0213, 0.230)
   - Camera F2: (16.4, -203.3, -230) -> (0.0164, 0.2033, 0.230)
@@ -104,5 +100,5 @@
   <!-- ====================================================================== -->
   <!-- IMU Sensor -->
-  <!-- Current connector/reference value: (0.0656, +0.091, 0.203)m.
+  <!-- Final May 2026 seed: imu_link origin (-0.01188, +0.12755, 0.23412)m.
        Encased MTi-30 AHRS device ID 0368xxxx: connector side is -X and exits
        aft, the unit is upside down, so +X is forward, +Y is starboard/right,
@@ -124,5 +120,5 @@
     <parent link="base_link"/>
     <child link="imu_link"/>
-    <origin xyz="0.0656 0.091 0.203" rpy="3.141592653589793 0 0"/>
+    <origin xyz="-0.01188 0.12755 0.23412" rpy="3.141592653589793 0 0"/>
   </joint>
   <gazebo>
@@ -141,5 +137,5 @@
   </gazebo>
   <!-- ====================================================================== -->
-  <!-- GPS/NavSat link (same position as IMU for now) -->
+  <!-- GPS/NavSat link near the IMU for now. -->
   <!-- ====================================================================== -->
   <link name="navsat_link">
@@ -152,14 +148,11 @@
     <parent link="base_link"/>
     <child link="navsat_link"/>
-    <origin xyz="0.0656 0.091 0.25" rpy="0 0 0"/>
+    <origin xyz="-0.01188 0.12755 0.28112" rpy="0 0 0"/>
   </joint>
   <!-- ====================================================================== -->
   <!-- Horizontal Lidar (lidar_h) -->
-  <!-- VLP-16 origin is sensor center. The cable is on -Y_lidar and exits
-       toward the stern, so the sensor frame is yawed -90 deg relative to the
-       boat. Relative to the current IMU cable/reference point, the lidar cable
-       is 3.72 mm forward, 7.15 mm left, and 35.64 mm higher; the VLP center is
-       another 50.86 mm forward from the cable side and 36.19 mm above the cable
-       exit. Corrected center -> ROS: (0.12018, +0.09815, 0.27483)m. -->
+  <!-- Final May 2026 seed. VLP-16 origin is sensor center. The cable is on
+       -Y_lidar and exits aft, so the sensor frame is yawed -90 deg relative to
+       base_link. Center -> ROS: (0.00000, +0.13000, 0.29654)m. -->
   <!-- ====================================================================== -->
   <!-- Lidar H mount pole -->
@@ -180,5 +173,5 @@
     <parent link="base_link"/>
     <child link="lidar_h_mount"/>
-    <origin xyz="0.12018 0.09815 0.16" rpy="0 0 0"/>
+    <origin xyz="0.00000 0.13000 0.16" rpy="0 0 0"/>
   </joint>
   <link name="lidar_h_link">
@@ -203,11 +196,10 @@
     <parent link="base_link"/>
     <child link="lidar_h_link"/>
-    <origin xyz="0.12018 0.09815 0.27483" rpy="0 0 -1.5707963267948966"/>
+    <origin xyz="0.00000 0.13000 0.29654" rpy="0 0 -1.5707963267948966"/>
   </joint>
   <!-- ====================================================================== -->
   <!-- Vertical Lidar (lidar_v) -->
-  <!-- Vertical VLP reference plane is 0.10298 m behind the lidar_h connector.
-       With lidar_v +Z aft and the VLP origin at sensor center, the center is
-       one radius forward from that plane: (0.01720, +0.126, 0.181)m. -->
+  <!-- Final May 2026 seed. Vertical VLP center -> ROS:
+       (-0.19003, +0.12234, 0.18068)m. -->
   <!-- Vertical VLP-16 frame: +X starboard/right, +Y up, +Z aft/stern. -->
   <!-- ====================================================================== -->
@@ -229,5 +221,5 @@
     <parent link="base_link"/>
     <child link="lidar_v_mount"/>
-    <origin xyz="0.01720 0.126 0.11" rpy="0 0 0"/>
+    <origin xyz="-0.19003 0.12234 0.11" rpy="0 0 0"/>
   </joint>
   <link name="lidar_v_link">
@@ -252,5 +244,5 @@
     <parent link="base_link"/>
     <child link="lidar_v_link"/>
-    <origin xyz="0.01720 0.126 0.181" rpy="1.5707963267948966 0 -1.5707963267948966"/>
+    <origin xyz="-0.19003 0.12234 0.18068" rpy="1.5707963267948966 0 -1.5707963267948966"/>
   </joint>
   <!-- ====================================================================== -->

File: urdf/ig_handle_sensors.urdf.xacro (robot description, xacro)
@@ -19,10 +19,7 @@
   <!-- ====================================================================== -->
   <!-- Lidar H (Horizontal) -->
-  <!-- VLP-16 origin is sensor center. The cable is on -Y_lidar and exits
-       toward the stern, so the sensor frame is yawed -90 deg relative to the
-       boat. Relative to the current IMU cable/reference point, the lidar cable
-       is 3.72 mm forward, 7.15 mm left, and 35.64 mm higher; the VLP center is
-       another 50.86 mm forward from the cable side and 36.19 mm above the cable
-       exit. Corrected center -> ROS: (0.12018, 0.09815, 0.27483)m. -->
+  <!-- Final May 2026 seed. VLP-16 origin is sensor center. The cable is on
+       -Y_lidar and exits aft, so the sensor frame is yawed -90 deg relative to
+       base_link. Center -> ROS: (0.00000, 0.13000, 0.29654)m. -->
   <!-- Velodyne VLP-16 model: 16 channels, 360 degree sweep, 10 Hz at 600 RPM. -->
   <!-- ====================================================================== -->
@@ -41,5 +38,5 @@
     <parent link="base_link"/>
     <child link="lidar_h_mount"/>
-    <origin xyz="0.12018 0.09815 0.16" rpy="0 0 0"/>
+    <origin xyz="0.00000 0.13000 0.16" rpy="0 0 0"/>
   </joint>
   <link name="lidar_h_link">
@@ -56,5 +53,5 @@
     <parent link="base_link"/>
     <child link="lidar_h_link"/>
-    <origin xyz="0.12018 0.09815 0.27483" rpy="0 0 -1.5707963267948966"/>
+    <origin xyz="0.00000 0.13000 0.29654" rpy="0 0 -1.5707963267948966"/>
   </joint>
   <gazebo reference="lidar_h_link">
@@ -102,7 +99,6 @@
   <!-- ====================================================================== -->
   <!-- Lidar V (Vertical) -->
-  <!-- Vertical VLP reference plane is 0.10298 m behind the lidar_h connector.
-       With lidar_v +Z aft and the VLP origin at sensor center, the center is
-       one radius forward from that plane: (0.01720, 0.126, 0.181)m. -->
+  <!-- Final May 2026 seed. Vertical VLP center -> ROS:
+       (-0.19003, 0.12234, 0.18068)m. -->
   <!-- Vertical VLP-16 frame: +X starboard/right, +Y up, +Z aft/stern. -->
   <!-- ====================================================================== -->
@@ -121,5 +117,5 @@
     <parent link="base_link"/>
     <child link="lidar_v_mount"/>
-    <origin xyz="0.01720 0.126 0.11" rpy="0 0 0"/>
+    <origin xyz="-0.19003 0.12234 0.11" rpy="0 0 0"/>
   </joint>
   <link name="lidar_v_link">
@@ -136,5 +132,5 @@
     <parent link="base_link"/>
     <child link="lidar_v_link"/>
-    <origin xyz="0.01720 0.126 0.181" rpy="1.5707963267948966 0 -1.5707963267948966"/>
+    <origin xyz="-0.19003 0.12234 0.18068" rpy="1.5707963267948966 0 -1.5707963267948966"/>
   </joint>
   <gazebo reference="lidar_v_link">
@@ -365,5 +361,5 @@
   <!-- ====================================================================== -->
   <!-- IMU Visual (for debugging) -->
-  <!-- Current connector/reference value: (0.0656, 0.091, 0.203)m.
+  <!-- Final May 2026 seed: imu_link origin (-0.01188, 0.12755, 0.23412)m.
        Encased MTi-30 AHRS device ID 0368xxxx: connector side is -X and exits
        aft, the unit is upside down, so +X is forward, +Y is starboard/right,
@@ -385,5 +381,5 @@
     <parent link="base_link"/>
     <child link="debug_extra_link"/>
-    <origin xyz="0.0656 0.091 0.203" rpy="3.141592653589793 0 0"/>
+    <origin xyz="-0.01188 0.12755 0.23412" rpy="3.141592653589793 0 0"/>
   </joint>
   <gazebo>

Commit message: Use canonical Heron sensor geometry

File: urdf/heron_sim.urdf.xacro (robot description, xacro)
@@ -8,8 +8,10 @@
   - lidar_v VLP-16 origin: (-0.19003, +0.12234, 0.18068), roll 90 deg + yaw -90 deg
   - imu_link origin: (-0.01188, +0.12755, 0.23412), roll 180 deg
-  - Camera F1: (16.4, -21.3, -230) -> (0.0164, 0.0213, 0.230)
-  - Camera F2: (16.4, -203.3, -230) -> (0.0164, 0.2033, 0.230)
-  - Camera F3: (16.4, -21.3, -230) -> (0.0164, 0.0213, 0.230), upward
-  - Camera F4: (16.4, -203.3, -230) -> (0.0164, 0.2033, 0.230), upward
+  - Camera F1 optical origin: (0.02445, 0.04035, 0.22909), forward center-ish
+  - Camera F2 optical origin: (0.02445, 0.21966, 0.22909), forward port
+  - Camera F3 optical origin: (0.02445, 0.26652, 0.18339), upward port
+  - Camera F4 optical origin: (0.02445, -0.00652, 0.18339), upward center-ish
+  This standalone URDF is legacy; the active simulator uses
+  ig_handle_benchmark plus ig_handle_sensors.urdf.xacro.
 -->
 <robot name="heron_sim" xmlns:xacro="http://www.ros.org/wiki/xacro">
@@ -152,7 +154,6 @@
   <!-- ====================================================================== -->
   <!-- Horizontal Lidar (lidar_h) -->
-  <!-- Final May 2026 seed. VLP-16 origin is sensor center. The cable is on
-       -Y_lidar and exits aft, so the sensor frame is yawed -90 deg relative to
-       base_link. Center -> ROS: (0.00000, +0.13000, 0.29654)m. -->
+  <!-- Seed mirrors slam_grande/config/sensors/heron_sensor_suite.yaml. -->
+  <!-- Horizontal VLP-16: +X starboard, +Y bow, +Z up. -->
   <!-- ====================================================================== -->
   <!-- Lidar H mount pole -->
@@ -200,7 +201,6 @@
   <!-- ====================================================================== -->
   <!-- Vertical Lidar (lidar_v) -->
-  <!-- Final May 2026 seed. Vertical VLP center -> ROS:
-       (-0.19003, +0.12234, 0.18068)m. -->
-  <!-- Vertical VLP-16 frame: +X starboard/right, +Y up, +Z aft/stern. -->
+  <!-- Vertical VLP-16: +X starboard, +Y up, +Z aft. Keep the runtime
+       ownership edge as lidar_h_link -> lidar_v_link. -->
   <!-- ====================================================================== -->
   <!-- Lidar V mount pole -->
@@ -242,7 +242,7 @@
   </link>
   <joint name="lidar_v_joint" type="fixed">
-    <parent link="base_link"/>
+    <parent link="lidar_h_link"/>
     <child link="lidar_v_link"/>
-    <origin xyz="-0.19003 0.12234 0.18068" rpy="1.5707963267948966 0 -1.5707963267948966"/>
+    <origin xyz="0.00766 -0.19003 -0.11586" rpy="1.5707963267948966 0 0"/>
   </joint>
   <!-- ====================================================================== -->
@@ -265,9 +265,8 @@
     <parent link="base_link"/>
     <child link="camera_mount"/>
-    <origin xyz="0.0164 0.1 0.13" rpy="0 0 0"/>
-  </joint>
-  <!-- ====================================================================== -->
-  <!-- Camera F1 (forward left-side) -->
-  <!-- User: (16.4, -21.3, -230)mm -> ROS: (0.0164, +0.0213, 0.230)m -->
+    <origin xyz="0.02445 0.13000 0.13000" rpy="0 0 0"/>
+  </joint>
+  <!-- ====================================================================== -->
+  <!-- Camera F1 (forward center-ish) -->
   <!-- ====================================================================== -->
   <link name="F1">
@@ -291,5 +290,5 @@
     <parent link="base_link"/>
     <child link="F1"/>
-    <origin xyz="0.0164 0.0213 0.230" rpy="0 0 0"/>
+    <origin xyz="0.02445 0.04035 0.22909" rpy="0 0 0"/>
   </joint>
   <!-- Camera F1 optical frame -->
@@ -298,10 +297,9 @@
     <parent link="F1"/>
     <child link="F1_optical"/>
-    <origin xyz="0 0 0" rpy="-1.5708 0 -1.5708"/>
+    <origin xyz="0 0 0" rpy="-1.5707963267948966 0 -1.5707963267948966"/>
   </joint>
   <xacro:if value="$(optenv HERON_CAMERA_F2 0)">
     <!-- ====================================================================== -->
-    <!-- Camera F2 (forward center-ish) -->
-    <!-- User: (16.4, -203.3, -230)mm -> ROS: (0.0164, +0.2033, 0.230)m -->
+    <!-- Camera F2 (forward port) -->
     <!-- ====================================================================== -->
     <link name="F2">
@@ -325,5 +323,5 @@
       <parent link="base_link"/>
       <child link="F2"/>
-      <origin xyz="0.0164 0.2033 0.230" rpy="0 0 0"/>
+      <origin xyz="0.02445 0.21966 0.22909" rpy="0 0 0"/>
     </joint>
     <!-- Camera F2 optical frame -->
@@ -332,11 +330,10 @@
       <parent link="F2"/>
       <child link="F2_optical"/>
-      <origin xyz="0 0 0" rpy="-1.5708 0 -1.5708"/>
+      <origin xyz="0 0 0" rpy="-1.5707963267948966 0 -1.5707963267948966"/>
     </joint>
   </xacro:if>
   <xacro:if value="$(optenv HERON_CAMERA_F3 0)">
     <!-- ====================================================================== -->
-    <!-- Camera F3 (upward left-side) -->
-    <!-- User: (16.4, -21.3, -230)mm -> ROS: (0.0164, +0.0213, 0.230)m -->
+    <!-- Camera F3 (upward port) -->
     <!-- ====================================================================== -->
     <link name="F3">
@@ -360,5 +357,5 @@
       <parent link="base_link"/>
       <child link="F3"/>
-      <origin xyz="0.0164 0.0213 0.230" rpy="0 -1.5708 0"/>
+      <origin xyz="0.02445 0.26652 0.18339" rpy="0 -1.5707963267948966 0"/>
     </joint>
     <!-- Camera F3 optical frame -->
@@ -367,10 +364,9 @@
       <parent link="F3"/>
       <child link="F3_optical"/>
-      <origin xyz="0 0 0" rpy="-1.5708 0 -1.5708"/>
+      <origin xyz="0 0 0" rpy="-1.5707963267948966 0 -1.5707963267948966"/>
     </joint>
   </xacro:if>
   <!-- ====================================================================== -->
   <!-- Camera F4 (upward center-ish) -->
-  <!-- User: (16.4, -203.3, -230)mm -> ROS: (0.0164, +0.2033, 0.230)m -->
   <!-- ====================================================================== -->
   <link name="F4">
@@ -394,5 +390,5 @@
     <parent link="base_link"/>
     <child link="F4"/>
-    <origin xyz="0.0164 0.2033 0.230" rpy="0 -1.5708 0"/>
+    <origin xyz="0.02445 -0.00652 0.18339" rpy="0 -1.5707963267948966 0"/>
   </joint>
   <!-- Camera F4 optical frame -->
@@ -401,5 +397,5 @@
     <parent link="F4"/>
     <child link="F4_optical"/>
-    <origin xyz="0 0 0" rpy="-1.5708 0 -1.5708"/>
+    <origin xyz="0 0 0" rpy="-1.5707963267948966 0 -1.5707963267948966"/>
   </joint>
   <!-- ====================================================================== -->

File: urdf/ig_handle_sensors.urdf.xacro (robot description, xacro)
@@ -19,7 +19,7 @@
   <!-- ====================================================================== -->
   <!-- Lidar H (Horizontal) -->
-  <!-- Final May 2026 seed. VLP-16 origin is sensor center. The cable is on
-       -Y_lidar and exits aft, so the sensor frame is yawed -90 deg relative to
-       base_link. Center -> ROS: (0.00000, 0.13000, 0.29654)m. -->
+  <!-- Sensor origins come from slam_grande/config/sensors/heron_sensor_suite.yaml
+       via HERON_* environment variables exported by ig_handle_benchmark. -->
+  <!-- Horizontal VLP-16: +X starboard, +Y bow, +Z up. -->
   <!-- Velodyne VLP-16 model: 16 channels, 360 degree sweep, 10 Hz at 600 RPM. -->
   <!-- ====================================================================== -->
@@ -38,5 +38,5 @@
     <parent link="base_link"/>
     <child link="lidar_h_mount"/>
-    <origin xyz="0.00000 0.13000 0.16" rpy="0 0 0"/>
+    <origin xyz="$(optenv HERON_LIDAR_H_MOUNT_XYZ)" rpy="0 0 0"/>
   </joint>
   <link name="lidar_h_link">
@@ -53,5 +53,5 @@
     <parent link="base_link"/>
     <child link="lidar_h_link"/>
-    <origin xyz="0.00000 0.13000 0.29654" rpy="0 0 -1.5707963267948966"/>
+    <origin xyz="$(optenv HERON_LIDAR_H_XYZ)" rpy="$(optenv HERON_LIDAR_H_RPY)"/>
   </joint>
   <gazebo reference="lidar_h_link">
@@ -99,7 +99,6 @@
   <!-- ====================================================================== -->
   <!-- Lidar V (Vertical) -->
-  <!-- Final May 2026 seed. Vertical VLP center -> ROS:
-       (-0.19003, 0.12234, 0.18068)m. -->
-  <!-- Vertical VLP-16 frame: +X starboard/right, +Y up, +Z aft/stern. -->
+  <!-- Vertical VLP-16: +X starboard, +Y up, +Z aft. Runtime TF ownership is
+       lidar_h_link -> lidar_v_link; the mount visual remains in base_link. -->
   <!-- ====================================================================== -->
   <!-- Mount pole for Lidar V -->
@@ -117,5 +116,5 @@
     <parent link="base_link"/>
     <child link="lidar_v_mount"/>
-    <origin xyz="-0.19003 0.12234 0.11" rpy="0 0 0"/>
+    <origin xyz="$(optenv HERON_LIDAR_V_MOUNT_XYZ)" rpy="0 0 0"/>
   </joint>
   <link name="lidar_v_link">
@@ -130,7 +129,7 @@
   </link>
   <joint name="lidar_v_joint" type="fixed">
-    <parent link="base_link"/>
+    <parent link="lidar_h_link"/>
     <child link="lidar_v_link"/>
-    <origin xyz="-0.19003 0.12234 0.18068" rpy="1.5707963267948966 0 -1.5707963267948966"/>
+    <origin xyz="$(optenv HERON_LIDAR_V_XYZ)" rpy="$(optenv HERON_LIDAR_V_RPY)"/>
   </joint>
   <gazebo reference="lidar_v_link">
@@ -250,5 +249,5 @@
     <parent link="base_link"/>
     <child link="camera_mount"/>
-    <origin xyz="0.0164 0.1 0.13" rpy="0 0 0"/>
+    <origin xyz="$(optenv HERON_CAMERA_MOUNT_XYZ)" rpy="0 0 0"/>
   </joint>
   <xacro:macro name="ig_handle_forge_camera"
@@ -273,5 +272,5 @@
       <parent link="${id}"/>
       <child link="${id}_optical"/>
-      <origin xyz="0 0 0" rpy="-1.5708 0 -1.5708"/>
+      <origin xyz="0 0 0" rpy="-1.5707963267948966 0 -1.5707963267948966"/>
     </joint>
     <gazebo reference="${id}">
@@ -321,8 +320,8 @@
   <xacro:if value="$(optenv HERON_CAMERA_F1 1)">
     <xacro:ig_handle_forge_camera id="F1"
-                                  xyz="0.0164 0.0213 0.230"
-                                  rpy="0 0 0"
+                                  xyz="$(optenv HERON_CAMERA_F1_XYZ)"
+                                  rpy="$(optenv HERON_CAMERA_F1_RPY)"
                                   topic_suffix="f1"
-                                  camera_name="forward_left"
+                                  camera_name="forward_center"
                                   distortion_k1="-0.0100"
                                   distortion_k2="0.0030"
@@ -331,8 +330,8 @@
   <xacro:if value="$(optenv HERON_CAMERA_F2 0)">
     <xacro:ig_handle_forge_camera id="F2"
-                                  xyz="0.0164 0.2033 0.230"
-                                  rpy="0 0 0"
+                                  xyz="$(optenv HERON_CAMERA_F2_XYZ)"
+                                  rpy="$(optenv HERON_CAMERA_F2_RPY)"
                                   topic_suffix="f2"
-                                  camera_name="forward_center"
+                                  camera_name="forward_left"
                                   distortion_k1="-0.0090"
                                   distortion_k2="0.0028"
@@ -341,6 +340,6 @@
   <xacro:if value="$(optenv HERON_CAMERA_F3 0)">
     <xacro:ig_handle_forge_camera id="F3"
-                                  xyz="0.0164 0.0213 0.230"
-                                  rpy="0 -1.5708 0"
+                                  xyz="$(optenv HERON_CAMERA_F3_XYZ)"
+                                  rpy="$(optenv HERON_CAMERA_F3_RPY)"
                                   topic_suffix="f3"
                                   camera_name="upward_left"
@@ -351,6 +350,6 @@
   <xacro:if value="$(optenv HERON_CAMERA_F4 1)">
     <xacro:ig_handle_forge_camera id="F4"
-                                  xyz="0.0164 0.2033 0.230"
-                                  rpy="0 -1.5708 0"
+                                  xyz="$(optenv HERON_CAMERA_F4_XYZ)"
+                                  rpy="$(optenv HERON_CAMERA_F4_RPY)"
                                   topic_suffix="f4"
                                   camera_name="upward_center"
@@ -361,5 +360,5 @@
   <!-- ====================================================================== -->
   <!-- IMU Visual (for debugging) -->
-  <!-- Final May 2026 seed: imu_link origin (-0.01188, 0.12755, 0.23412)m.
+  <!-- IMU pose comes from the canonical sensor suite through HERON_IMU_*.
        Encased MTi-30 AHRS device ID 0368xxxx: connector side is -X and exits
        aft, the unit is upside down, so +X is forward, +Y is starboard/right,
@@ -381,5 +380,5 @@
     <parent link="base_link"/>
     <child link="debug_extra_link"/>
-    <origin xyz="-0.01188 0.12755 0.23412" rpy="3.141592653589793 0 0"/>
+    <origin xyz="$(optenv HERON_IMU_XYZ)" rpy="$(optenv HERON_IMU_RPY)"/>
   </joint>
   <gazebo>
