Commit message: Simplify Heron simulator assets

File: urdf/sensors.urdf.xacro (robot description, xacro)
@@ -2,8 +2,7 @@
 <robot xmlns:xacro="http://www.ros.org/wiki/xacro">
   <!-- ====================================================================== -->
-  <!-- IG Handle Sensors Configuration                                        -->
-  <!-- User coordinate frame: x-forward, y-right, z-down                      -->
-  <!-- ROS coordinate frame: x-forward, y-left, z-up                          -->
-  <!-- Conversion: negate Y and Z                                             -->
+  <!-- IG Handle simulator sensor add-on. All sensor frame and mount poses
+       come from ig_handle/config/sensors/sensor_frames.yaml through
+       ig_handle/scripts/frames/export.py and HERON_* environment variables. -->
   <!-- ====================================================================== -->
   <!-- Material Definitions -->
@@ -19,5 +18,5 @@
   <!-- ====================================================================== -->
   <!-- Lidar H (Horizontal) -->
-  <!-- Sensor origins come from slam_grande/config/sensors/heron_sensor_suite.yaml
+  <!-- Sensor origins come from ig_handle/config/sensors/sensor_frames.yaml
        via HERON_* environment variables exported by ig_handle_benchmark. -->
   <!-- Horizontal VLP-16: +X starboard, +Y bow, +Z up. -->
@@ -38,5 +37,5 @@
     <parent link="base_link"/>
     <child link="lidar_h_mount"/>
-    <origin xyz="$(optenv HERON_LIDAR_H_MOUNT_XYZ)" rpy="0 0 0"/>
+    <origin xyz="$(optenv HERON_LIDAR_H_MOUNT_XYZ)" rpy="$(optenv HERON_LIDAR_H_MOUNT_RPY)"/>
   </joint>
   <link name="lidar_h_link">
@@ -116,5 +115,5 @@
     <parent link="base_link"/>
     <child link="lidar_v_mount"/>
-    <origin xyz="$(optenv HERON_LIDAR_V_MOUNT_XYZ)" rpy="0 0 0"/>
+    <origin xyz="$(optenv HERON_LIDAR_V_MOUNT_XYZ)" rpy="$(optenv HERON_LIDAR_V_MOUNT_RPY)"/>
   </joint>
   <link name="lidar_v_link">
@@ -177,5 +176,5 @@
   <!-- ====================================================================== -->
   <!-- Sonar -->
-  <!-- Imagenex DT100 profile model. User: (0, 0, 80)mm -> ROS: (0, 0, -0.08)m. -->
+  <!-- Imagenex DT100 profile model. Pose comes from sensor_frames.yaml. -->
   <!-- The acoustic +X axis is pitched down into ROS -Z. The ray fan models the -->
   <!-- 480-beam, 120 degree cross-track profile. The physical 3 degree along-track -->
@@ -196,5 +195,5 @@
     <parent link="base_link"/>
     <child link="sonar_link"/>
-    <origin xyz="0 0 -0.08" rpy="0 1.5708 0"/>
+    <origin xyz="$(optenv HERON_SONAR_XYZ)" rpy="$(optenv HERON_SONAR_RPY)"/>
   </joint>
   <gazebo reference="sonar_link">
@@ -223,5 +222,5 @@
       </ray>
       <plugin name="sonar_plugin" filename="libgazebo_ros_velodyne_laser.so">
-        <topicName>/sensors/sonar/scan</topicName>
+        <topicName>$(optenv HERON_SIM_SONAR_RAY_TOPIC /sim/sensors/sonar/multibeam_points)</topicName>
         <frameName>sonar_link</frameName>
         <min_range>0.5</min_range>
@@ -249,8 +248,8 @@
     <parent link="base_link"/>
     <child link="camera_mount"/>
-    <origin xyz="$(optenv HERON_CAMERA_MOUNT_XYZ)" rpy="0 0 0"/>
+    <origin xyz="$(optenv HERON_CAMERA_MOUNT_XYZ)" rpy="$(optenv HERON_CAMERA_MOUNT_RPY)"/>
   </joint>
   <xacro:macro name="ig_handle_forge_camera"
-               params="id xyz rpy topic_suffix camera_name distortion_k1 distortion_k2 distortion_k3">
+               params="id xyz rpy optical_rpy topic_suffix camera_name distortion_k1 distortion_k2 distortion_k3">
     <link name="${id}">
       <visual>
@@ -272,5 +271,5 @@
       <parent link="${id}"/>
       <child link="${id}_optical"/>
-      <origin xyz="0 0 0" rpy="-1.5707963267948966 0 -1.5707963267948966"/>
+      <origin xyz="0 0 0" rpy="${optical_rpy}"/>
     </joint>
     <gazebo reference="${id}">
@@ -323,4 +322,5 @@
                                   xyz="$(optenv HERON_CAMERA_F1_XYZ)"
                                   rpy="$(optenv HERON_CAMERA_F1_RPY)"
+                                  optical_rpy="$(optenv HERON_CAMERA_FORWARD_OPTICAL_RPY)"
                                   topic_suffix="f1"
                                   camera_name="forward_starboard"
@@ -333,4 +333,5 @@
                                   xyz="$(optenv HERON_CAMERA_F2_XYZ)"
                                   rpy="$(optenv HERON_CAMERA_F2_RPY)"
+                                  optical_rpy="$(optenv HERON_CAMERA_FORWARD_OPTICAL_RPY)"
                                   topic_suffix="f2"
                                   camera_name="forward_port"
@@ -339,8 +340,9 @@
                                   distortion_k3="-0.0019"/>
   </xacro:if>
-  <xacro:if value="$(optenv HERON_CAMERA_F3 0)">
+  <xacro:if value="$(optenv HERON_CAMERA_F3 1)">
     <xacro:ig_handle_forge_camera id="F3"
                                   xyz="$(optenv HERON_CAMERA_F3_XYZ)"
                                   rpy="$(optenv HERON_CAMERA_F3_RPY)"
+                                  optical_rpy="$(optenv HERON_CAMERA_UPWARD_OPTICAL_RPY)"
                                   topic_suffix="f3"
                                   camera_name="upward_port"
@@ -353,4 +355,5 @@
                                   xyz="$(optenv HERON_CAMERA_F4_XYZ)"
                                   rpy="$(optenv HERON_CAMERA_F4_RPY)"
+                                  optical_rpy="$(optenv HERON_CAMERA_UPWARD_OPTICAL_RPY)"
                                   topic_suffix="f4"
                                   camera_name="upward_starboard"
@@ -361,5 +364,5 @@
   <!-- ====================================================================== -->
   <!-- IMU Visual (for debugging) -->
-  <!-- IMU pose comes from the canonical sensor suite through HERON_IMU_*.
+  <!-- IMU pose comes from the canonical sensor frame config through HERON_IMU_*.
        Encased MTi-30 AHRS device ID 0368xxxx: connector side is -X and exits
        aft, the unit is upside down, so +X is forward, +Y is starboard/right,
