Commit message: Add descriptor-driven acoustic marker scenario

File: urdf/sensors.urdf.xacro (robot description, xacro)
@@ -182,5 +182,5 @@
   <!-- one profile slice per ping. -->
   <!-- ====================================================================== -->
-  <link name="sonar_link">
+  <link name="dt100_link">
     <visual>
       <geometry><cylinder radius="0.03" length="0.05"/></geometry>
@@ -192,11 +192,11 @@
     </inertial>
   </link>
-  <joint name="sonar_joint" type="fixed">
-    <parent link="base_link"/>
-    <child link="sonar_link"/>
-    <origin xyz="$(optenv HERON_SONAR_XYZ)" rpy="$(optenv HERON_SONAR_RPY)"/>
-  </joint>
-  <gazebo reference="sonar_link">
-    <sensor type="ray" name="sonar">
+  <joint name="dt100_joint" type="fixed">
+    <parent link="base_link"/>
+    <child link="dt100_link"/>
+    <origin xyz="$(optenv HERON_DT100_XYZ)" rpy="$(optenv HERON_DT100_RPY)"/>
+  </joint>
+  <gazebo reference="dt100_link">
+    <sensor type="ray" name="dt100">
       <update_rate>20</update_rate>
       <ray>
@@ -206,5 +206,6 @@
                <resolution>1</resolution>
                <min_angle>-1.047198</min_angle>
-               <max_angle>1.047198</max_angle>
+               <!-- 480 documented 0.25-degree 83P beam centers: -60 to +59.75 deg. -->
+               <max_angle>1.042834</max_angle>
             </horizontal>
             <vertical>
@@ -223,5 +224,5 @@
       <plugin name="sonar_plugin" filename="libgazebo_ros_velodyne_laser.so">
         <topicName>$(optenv HERON_SIM_SONAR_RAY_TOPIC /sim/sensors/sonar/multibeam_points)</topicName>
-        <frameName>sonar_link</frameName>
+        <frameName>dt100_link</frameName>
         <min_range>0.5</min_range>
         <max_range>100.0</max_range>
@@ -231,4 +232,21 @@
       </plugin>
     </sensor>
+  </gazebo>
+  <link name="ping360_link">
+    <visual>
+      <geometry><cylinder radius="0.03" length="0.05"/></geometry>
+      <material name="sensor_blue"/>
+    </visual>
+    <inertial>
+      <mass value="0.01"/>
+      <inertia ixx="0.0001" ixy="0" ixz="0" iyy="0.0001" iyz="0" izz="0.0001"/>
+    </inertial>
+  </link>
+  <joint name="ping360_joint" type="fixed">
+    <parent link="base_link"/>
+    <child link="ping360_link"/>
+    <origin xyz="$(optenv HERON_PING360_XYZ)" rpy="$(optenv HERON_PING360_RPY)"/>
+  </joint>
+  <gazebo reference="ping360_link">
     <!-- Separate full-circle environment sampler for the canonical Ping360
          simulator. It does not fabricate vendor wire packets: the simulator
@@ -259,5 +277,5 @@
       <plugin name="ping360_environment_plugin" filename="libgazebo_ros_velodyne_laser.so">
         <topicName>$(optenv HERON_SIM_PING360_RAY_TOPIC /sim/sensors/sonar/ping360_points)</topicName>
-        <frameName>sonar_link</frameName>
+        <frameName>ping360_link</frameName>
         <min_range>0.5</min_range>
         <max_range>100.0</max_range>
